File: sim/core-vdd-rail/core-vdd-rail.kicad_sch (KiCad schematic)
At the start: 66 parts, among them Q1 q-mosfet-nmos-dgs, Q2 q-mosfet-nmos-dgs

Commit message: Further elaboration of the USB / power module schematics.
Parts:
- added CFB1, CSS1, C_PLANE4, C_PLANE5: ${SIM.PARAMS}, restall-generic-capacitors:unpolarised-nominal-0402-1005, symbol restall-generic-capacitors:capacitor-unpolarised
- added RFB1, RFB2: ${SIM.PARAMS}, restall-generic-resistors:nominal-0402-1005, symbol restall-generic-resistors:resistor
- added U1: TPS62851?DRLR, restall-manufacturer-ti:SOT-583-8, symbol restall-manufacturer-ti:TPS62851?DRLR
Connections:
- net 0: now also CSS1.2, C_PLANE4.2, C_PLANE5.2, RFB2.1, U1.6 (PG), U1.8 (GND)
- net VIN: now also U1.1 (V_{IN}), U1.2 (EN), U1.3 (MODE)
- net VSW: now also CFB1.1, RFB1.2, U1.7 (SW)
- net V_HSD: now also C_PLANE4.1
- net V_LSD: now also C_PLANE5.1
- new net: CSS1.1, U1.4 (SS_TR)
- new net: CFB1.2, RFB1.1, RFB2.2, U1.5 (FB)
Other:
- note added: ".param pwmDead=4n"
- note added: ".param pwmPulseTw={pwmDutyCycle/pwmFrequencyHz-pwmTr}"
- note added: "JLC04161H-7628 (economical fab) Prepreg thickness is 0.2104mm C = 0.42pF / 10mm^{2}, 0.84pF / 20mm^{2}, 420pF / 100mm^{2}, etc. JLC04161H-3313 (non-economical fab) Prepreg thickness is 0.0994mm C = 0.89pF / 10mm^{2}, 1.78pF / 20mm^{2}, etc."
- note added: "The ripple on VIN is horrendous and the voltage on VSW violates the 10V absolute maximum. However, TI Webench simulations work alright but don't have the parasitics. I think the best thing is simply to build this as the simulation with parasitics is a time-sink - at least I have some ballpark figures for current ratings / limits, etc."
- note added: "Too many discontinuities in the TI model - disabled from simulation."
- note removed: ".param pwmPulseTw={pwmDutyCycle/pwmFrequencyHz-1n}"
- note removed: "TODO: THE RIPPLE ON VIN NEEDS TO BE SORTED - IT'S HORRENDOUS ! MAINLY ESL OF CAPS BY THE LOOKS."
