File: sim/msf-front-end/msf-front-end.kicad_sch (KiCad schematic)
At the start: 48 parts, among them K1 TMUX1511, K2 TMUX1511, K3 TMUX1511, K4 TMUX1511, K5 TMUX1511, K6 TMUX1511, K7 TMUX1511, K8 TMUX1511, U1 MCP6486, U2 MCP6486, U3 MCP6486, X1 60kHz, X2 60kHz, X3 60kHz

Commit message: Started to explore active filtering rather than using crystals for the MSF front-end.
Parts:
- added C11, Ca1, Ca2, Ca3, Ca4, Ca6, Col1: ${SIM.PARAMS}, restall-generic-capacitors:unpolarised-nominal-0402-1005, symbol restall-generic-capacitors:capacitor-unpolarised
- added Eol1: ESOURCE, symbol Simulation_SPICE:ESOURCE
- added R16, R17, R18, R19, Ra1, Ra2, Ra3, Ra4, Ra5, Ra6, Ra7, Ra8, Rol1: ${SIM.PARAMS}, restall-generic-resistors:nominal-0402-1005, symbol restall-generic-resistors:resistor
- added U4, U5, U6, Uol1: MCP6486, symbol Simulation_SPICE:OPAMP
- added Volac1, Vtst1: AC, symbol Simulation_SPICE:VSIN
- added Volvdd1: 3.6, symbol Simulation_SPICE:VDC
Connections:
- net GND: now also Col1.2, Eol1.2 (N-), Eol1.4 (C-), Ra2.1, Ra6.1, U4.5 (V-), U5.5 (V-), U6.5 (V-), Uol1.5 (V-), Volac1.2, Volvdd1.2
- net V_{dd+3.6V}: now also U4.4 (V+), U5.4 (V+), U6.4 (V+)
- net V_{in+2}: now also Ca3.2
- net V_{in-3}: now also C9.1
- net V_{out1}: now also Ra1.1
- net V_{out2}: now also Ra5.1; no longer C9.1
- net V_{out}: now also C11.1, R19.2; no longer C10.2, R15.2, U3.3
- net Vref_{+1.25V}: now also U4.1 (+), U5.1 (+), U6.1 (+), Vtst1.2
- net at C4.2, X1.1: now also C5.2, C6.2, C7.1, X1.2, X2.1, X2.2, X3.1, X3.2
- net V_{acsim}: now reaches Rmsf1.2, V2.1
- new net: Uol1.1 (+), Volac1.1
- new net: R16.2, R17.1, U5.2 (-)
- new net: R17.2, R18.1, U5.3
- new net: C11.2, R18.2
- new net: Ca1.2, Ca3.1, Ra7.2, U4.3
- new net: Eol1.1 (N+), Rol1.2
- new net: Ca4.1, Ca6.1, Ra5.2, Ra6.2
- new net: Ca1.1, Ca2.1, Ra1.2, Ra2.2
- new net: Ca2.2, Ra3.1, U4.2 (-)
- new net: Ra3.2, Ra7.1
- new net: Ca6.2, Ra4.1, U6.2 (-)
- new net: Ra4.2, Ra8.1
- new net: Uol1.4 (V+), Volvdd1.1
- new net: Col1.1, Rol1.1, Uol1.2 (-)
- new net V_{ol}: Eol1.3 (C+), Uol1.3
- new net V_{out3}: C10.2, R15.2, U3.3
- new net V_{out4}: Ca4.2, R16.1, R19.1, Ra8.2, U6.3
Other:
- note added: ".ac lin 100k 1 10Meg"
- note added: ".options Rshunt=10G gmin=0.1p"
- note added: "Open Loop Gain Measurement Rule of thumb (Op-Amps for Everyone, p461) - active filters need +40dB A_{o} headroom above filter response peak. The MCP6849 model does not vary A_{o} over V_{dd}, etc. so ensure an additional -6dB headroom to allow PVT variation."
- note added: "TODO: Better bridge ensuring equalised output delays - see Op-Amps for Everyone, p269"
- note added: "TODO: DON'T FORGET TO MONTE-CARLO OVER THE FILTER COMPONENTS..."
- note added: "TODO: WANTS TO BE RETURNED TO GND - IT IS POSSIBLE WITH MFB BUT NEEDS WORKING OUT..."
- note removed: "*options Rshunt=10G"
- note removed: ".ac lin 200k 1 10Meg"

Commit message: Tidied up the MSF front-end simulation.  Next step - Monte Carlo...
Parts:
- removed C10, C4, C5, C7, C9, Ca4, Ca6: ${SIM.PARAMS}, restall-generic-capacitors:unpolarised-nominal-0402-1005, symbol restall-generic-capacitors:capacitor-unpolarised
- removed R14, R15, R17, R7, Ra4, Ra5, Ra6, Ra8: ${SIM.PARAMS}, restall-generic-resistors:nominal-0402-1005, symbol restall-generic-resistors:resistor
- removed U6: MCP6486, symbol Simulation_SPICE:OPAMP
- removed Vtst1: AC, symbol Simulation_SPICE:VSIN
- removed X1, X2, X3: 60kHz, symbol Device:Crystal
- added Cfilt2_1, Cfilt2_2, Cref1, Cref2: ${SIM.PARAMS}, restall-generic-capacitors:unpolarised-nominal-0402-1005, symbol restall-generic-capacitors:capacitor-unpolarised
- added Radc2, Radc3, Radc4, Radc5, Radc6, Rfilt2_1, Rfilt2_2, Rfilt2_3, Rfilt2_4, Rref1, Rref2, Rref3, Rref4, Rsimforce1: ${SIM.PARAMS}, restall-generic-resistors:nominal-0402-1005, symbol restall-generic-resistors:resistor
- added U4, U7: MCP6486, symbol Simulation_SPICE:OPAMP
- added Vsimforce1: 1.25, symbol Simulation_SPICE:VDC
- V1: value 1.25 -> 2.5
- renumbered Ca3 to C4, C8 to C5, C11 to Cadc1, Ca1 to Cfilt1_1, Ca2 to Cfilt1_2, R11 to R10, R12 to R11, R13 to R12, R8 to R7, R9 to R8, R10 to R9, R16 to Radc1, R18 to Radc7, R19 to Radc8, Ra1 to Rfilt1_1, Ra2 to Rfilt1_2, Ra7 to Rfilt1_3, Ra3 to Rfilt1_4, U4 to U2, U2 to U3, U3 to U6
Connections:
- net V_{in-2} is gone; now on net V_{in-3}: C5.1, K5.14, R8.1, R9.1, U3.2 (-)
- net GND: now also V2.2, Cref1.1, Rfilt2_2.1, Rref2.1, U4.5 (V-), U7.5 (V-), Vsimforce1.2
- net V_{dd+3.6V}: now also U4.4 (V+), U7.4 (V+)
- net V_{in-3}: no longer U6.2 (-)
- net V_{out2}: now also C4.1, Cfilt1_1.2, Rfilt1_3.2, U2.3; no longer C5.2, K8.13, R12.2, U3.3
- net V_{out3}: now also C5.2, K8.13, R12.2, U3.3, Rfilt2_1.1; no longer U6.3
- net V_{out4}: now also C6.1, Cfilt2_1.2, Rfilt2_3.2, U4.3; no longer Radc1.1, Radc8.1
- net Vref_{+1.25V}: now also Rref4.2, Rsimforce1.2, U4.1 (+); no longer C6.1, Rvref1.1, U5.1 (+)
- net at C6.2: now also Radc1.1
- net at Radc1.2: now also U5.1 (+), Radc2.1; no longer U5.2 (-)
- net at Radc7.1, U5.3: now also Radc3.2, Radc5.2
- net V_{adc+}: now reaches Cadc1.2, Radc7.2
- net at Rvref1.2, V1.1: no longer V2.2
- net V_{in+2} renamed V_{in+3}
- net V_{out} renamed V_{adc-}
- new net: Radc2.2, Radc4.2, Radc6.2, Radc8.1, U6.3
- new net: Cfilt2_1.1, Cfilt2_2.1, Rfilt2_1.2, Rfilt2_2.2
- new net: Cref1.2, Rref1.1, Rref2.2, U7.1 (+)
- new net: Cref2.1, Rref3.1, U7.2 (-)
- new net: Cref2.2, Rref3.2, Rref4.1, U7.3
- new net: Radc5.1, Radc6.1, U6.2 (-)
- new net: Cfilt2_2.2, Rfilt2_4.1, U4.2 (-)
- new net: Radc3.1, Radc4.1, U5.2 (-)
- new net: Rsimforce1.1, Vsimforce1.1
- new net: Rfilt2_3.1, Rfilt2_4.2
- new net Vref_{+2.5V}: Rref1.2, Rvref1.1
Other:
- note added: "*tran 1u 500u 0"
- note added: ".nodeset v(/Vref+1.25V)=1.25"
- note added: ".param adcGainR=4.3k .param adcFeedbackR=10k"
- note added: ".param cVariationPercent=0.03 .param rVariationPercent=0.002"
- note added: "ADC Common-Mode Voltage Reference"
- note added: "Full-scale (~2.5V_{p-p} at the ADC) is ~730μV_{p-p} on maximum gain"
- note added: "MFB Bandpass (configurable as Deliyannis filter)"
- note added: "Single-Ended to Differential bridge ensuring equalised output delays - see Op-Amps for Everyone, p269."
- note removed: "*tran 1n 500u 0 10n"
- note removed: "TODO: Better bridge ensuring equalised output delays - see Op-Amps for Everyone, p269"
- note removed: "TODO: DON'T FORGET TO MONTE-CARLO OVER THE FILTER COMPONENTS..."
- note removed: "TODO: WANTS TO BE RETURNED TO GND - IT IS POSSIBLE WITH MFB BUT NEEDS WORKING OUT..."
- moved on the sheet: C4, C5, Cadc1, Cfilt1_1, Cfilt1_2, R10, R11, R12, R7, R8, R9, Radc1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

Commit message: Added a Monte-Carlo simulation to verify the MSF front-end over component variations.
Parts:
- renumbered C4 to C3, C6 to C4, C3 to Cpga1_1, C5 to Cpga2_1, R7 to R2, R2 to Rpga1_1, R3 to Rpga1_2, R4 to Rpga1_3, R5 to Rpga1_4, R6 to Rpga1_5, R8 to Rpga2_1, R9 to Rpga2_2, R10 to Rpga2_3, R11 to Rpga2_4, R12 to Rpga2_5
Other:
- note added: ".ac lin 10k 1 10Meg"
- note added: ".control setplot const let numberOfMonteCarloRuns = 0 let areFiltersAdjusted = 1 let arePgasAdjusted = 1 let isAdcBufferAdjusted = 1 let rngSeed = 1 + rnd(2^32-2) let Rfilt1 = 4.3k let Rfilt2 = 68 let Rfilt3 = 54.9k let Rfilt4 = 4.3k let Cfilt1 = 4.7n let Cfilt2 = 360p let Rpga1 = 100 let Rpga2 = 390 let Rpga3 = 1.24k let Rpga4 = 2.49k let Rpga5 = 4.99k let Cpga1 = 180p let CpgaDecoupling1 = 360p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"
- note added: "To run a Monte-Carlo simulation, set numberOfMonteCarloRuns > 0. The cWithTolerance5_0(x) function provides a uniform distribution of ±5% initial and ±1% temperature. The cWithTolerance2_0(x) function provides a uniform distribution of ±2% initial and ±1% temperature. The rWithTolerance1_0(x) function provides a uniform distribution of ±1% initial and ±1% temperature. The rWithTolerance0_1(x) fun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"
- note removed: ".ac lin 100k 1 10Meg"
- note removed: ".param cVariationPercent=0.03 .param rVariationPercent=0.002"

Commit message: Further refinement of the MSF Front-End and simulation.
Parts:
- added Cbypass2, Cbypass3, Cbypass4: 4.7u, restall-generic-capacitors:unpolarised-nominal-0402-1005, symbol restall-generic-capacitors:capacitor-unpolarised
- added Cbypass5, Cbypass6: 22u, restall-generic-capacitors:unpolarised-nominal-0805-2012, symbol restall-generic-capacitors:capacitor-unpolarised
- added L2: ${SIM.PARAMS}, symbol restall-generic-inductors:l-air
- Cbypass1: renamed from C2; value ${SIM.PARAMS} -> 4.7u
Connections:
- net GND: now also Cbypass2.2, Cbypass3.2, Cbypass4.2, Cbypass5.2, Cbypass6.2, L2.2 (P2)
- net V_{msf}: no longer Rmsf1.1
- net Vref_{+1.25V}: now also Cbypass2.1, Cbypass3.1, Cbypass4.1, Cbypass5.1, Cbypass6.1
- net V_{in+5}: now reaches Radc1.2, Radc2.1, U5.1 (+)
- net V_{in-6}: now reaches Radc5.1, Radc6.1, U6.2 (-)
- net V_{in-5}: now reaches Radc3.1, Radc4.1, U5.2 (-)
- new net: L2.1 (P1), Rmsf1.1
Other:
- note added: ".control setplot const let numberOfMonteCarloRuns = 20 let areFiltersAdjusted = 1 let arePgasAdjusted = 1 let isAdcBufferAdjusted = 1 let rngSeed = 1 + rnd(2^32-2) let Rfilt1 = 4.3k let Rfilt2 = 68 let Rfilt3 = 54.9k let Rfilt4 = 4.3k let Cfilt1 = 4.7n let Cfilt2 = 360p let Rpga1 = 100 let Rpga2 = 390 let Rpga3 = 1.24k let Rpga4 = 2.49k let Rpga5 = 4.99k let Cpga1 = 100p let CpgaDecoupling1 = 4.7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"
- note added: ".options Rshunt=10G Cshunt=0.1p gmin=0.1p"
- note added: ".param adcGainR=2.49k .param adcFeedbackR=2.49k"
- note added: "From V_{out4} to V_{adc+} is about -0.4dB; this loss is due to the filtering and must be factored into the maximum gain / smallest signal calculations to prevent hitting the rails and distortion; this is about 5% of the ADC at full-scale (205 codes)."
- note added: "Full-scale (~2.5V_{p-p} at the ADC) is ~1000μV_{p-p} on maximum gain"
- note added: "K L1 L2 0.999999"
- note removed: ".control setplot const let numberOfMonteCarloRuns = 0 let areFiltersAdjusted = 1 let arePgasAdjusted = 1 let isAdcBufferAdjusted = 1 let rngSeed = 1 + rnd(2^32-2) let Rfilt1 = 4.3k let Rfilt2 = 68 let Rfilt3 = 54.9k let Rfilt4 = 4.3k let Cfilt1 = 4.7n let Cfilt2 = 360p let Rpga1 = 100 let Rpga2 = 390 let Rpga3 = 1.24k let Rpga4 = 2.49k let Rpga5 = 4.99k let Cpga1 = 180p let CpgaDecoupling1 = 360p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"
- note removed: ".options Rshunt=10G gmin=0.1p"
- note removed: ".param adcGainR=4.3k .param adcFeedbackR=10k"
- note removed: "Full-scale (~2.5V_{p-p} at the ADC) is ~730μV_{p-p} on maximum gain"
- moved on the sheet: U6

Commit message: Ran the Monte-Carlo and transient simulations for the MSF front-end.  A decent first stab - noise analysis next.
Connections:
- net GND: no longer K1.A1, K2.A1, K3.A1, K4.A1, K5.A1, K6.A1, K7.A1, K8.A1
- net V_{dd+3.6V}: now also K1.A1, K2.A1, K3.A1, K4.A1, K5.A1, K6.A1, K7.A1, K8.A1
Other:
- note added: "*ac lin 10k 1 10Meg"
- note added: ".control setplot const let numberOfMonteCarloRuns = 0 let areFiltersAdjusted = 1 let arePgasAdjusted = 1 let isAdcBufferAdjusted = 1 let rngSeed = 1 + rnd(2^32-2) let Rfilt1 = 4.3k let Rfilt2 = 68 let Rfilt3 = 54.9k let Rfilt4 = 4.3k let Cfilt1 = 4.7n let Cfilt2 = 360p let Rpga1 = 100 let Rpga2 = 390 let Rpga3 = 1.24k let Rpga4 = 2.49k let Rpga5 = 4.99k let Cpga1 = 100p let CpgaDecoupling1 = 4.7n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"
- note added: ".nodeset v(/Vref+1.25V)=1.25 .nodeset v(/Vin+1)=1.25 .nodeset v(/Vin+3)=1.25 .nodeset v(/Vin+5)=1.25 .nodeset v(/Vin-5)=1.25 .nodeset v(/Vin-6)=1.25"
- note added: ".options Rshunt=10G Cshunt=0.1p gmin=0.1p reltol=0.01"
- note added: ".tran 200n 500u 0"
- note added: "For V2 transient simulation, set V=410u with maximum gain or V=1.55V with minimum gain"
- note added: "From V_{out4} to V_{adc+} is about -0.4dB; this loss is due to the filtering and must be factored into the maximum gain / smallest signal calculations to prevent hitting the rails and distortion; this is about 5% of the ADC at full-scale (205 codes). From transient analysis, around 410μV_{p-p} is the maximum input signal without significant distortion (around 2.344V_{p-p}), meaning about 6.3% hea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"
- note added: "Full-scale (~2.5V_{p-p} at the ADC) is ~410μV_{p-p} on maximum gain"
- note added: "Monte-Carlo on 100 runs for differential ADC voltage with maximum PGA gain: +81.5dB to +79.5dB @ 60kHz -16.9 to -18.5dB @ 180kHz About 15 bits Monte-Carlo on 100 runs for differential ADC voltage with minimum PGA gain: +10.5dB to +7.6dB @ 60kHz -74.6dB to -75.5dB @ 180kHz About 13 bits"
- note removed: "*tran 1u 500u 0"
- note removed: ".ac lin 10k 1 10Meg"
- note removed: ".control setplot const let numberOfMonteCarloRuns = 20 let areFiltersAdjusted = 1 let arePgasAdjusted = 1 let isAdcBufferAdjusted = 1 let rngSeed = 1 + rnd(2^32-2) let Rfilt1 = 4.3k let Rfilt2 = 68 let Rfilt3 = 54.9k let Rfilt4 = 4.3k let Cfilt1 = 4.7n let Cfilt2 = 360p let Rpga1 = 100 let Rpga2 = 390 let Rpga3 = 1.24k let Rpga4 = 2.49k let Rpga5 = 4.99k let Cpga1 = 100p let CpgaDecoupling1 = 4.7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"
- note removed: ".nodeset v(/Vref+1.25V)=1.25"
- note removed: ".options Rshunt=10G Cshunt=0.1p gmin=0.1p"
- note removed: "From V_{out4} to V_{adc+} is about -0.4dB; this loss is due to the filtering and must be factored into the maximum gain / smallest signal calculations to prevent hitting the rails and distortion; this is about 5% of the ADC at full-scale (205 codes)."
- note removed: "Full-scale (~2.5V_{p-p} at the ADC) is ~1000μV_{p-p} on maximum gain"
- moved on the sheet: Rmsf1, Rvdd1, Rvref1, V1, V2, V3

Commit message: Investigations around noise for the MSF front-end.  WIP.
Connections:
- net GND: now also K1.A1, K2.A1, K3.A1, K4.A1, K5.A1, K6.A1, K7.A1, K8.A1
- net V_{dd+3.6V}: no longer K1.A1, K2.A1, K3.A1, K4.A1, K5.A1, K6.A1, K7.A1, K8.A1
Other:
- note added: "*noise v(/Vadc+, /Vadc-) V2 lin 10k 1 10Meg"
- note added: "*tran 200n 500u 0"
- note added: ".control setplot const let isNoiseAnalysis = 1 let numberOfMonteCarloRuns = 0 let areFiltersAdjusted = 1 let arePgasAdjusted = 1 let isAdcBufferAdjusted = 1 let rngSeed = 1 + rnd(2^32-2) let Rfilt1 = 4.3k let Rfilt2 = 68 let Rfilt3 = 54.9k let Rfilt4 = 4.3k let Cfilt1 = 4.7n let Cfilt2 = 360p let Rpga1 = 100 let Rpga2 = 390 let Rpga3 = 1.24k let Rpga4 = 2.49k let Rpga5 = 4.99k let Cpga1 = 100p le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"
- note added: "Noise at the ADC is about 2.32μV/Hz^{-1} at 60kHz for minimum gain. Assuming a DFT with 1024 bins and an ADC sampling at 240kHz (about 5ms latency), each bin has a bandwidth of 235Hz. Using a filter shape factor of 1.57 we get: 2.32μV/Hz^{-1} * sqrt(235 * 1.57) = 44.6μV_{rms} That equates to just over half an LSb for 15-bit sampling. We can of course decrease the bin with at the expense of latenc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"
- note added: "To run a Monte-Carlo simulation, set isNoiseAnalysis=0 and numberOfMonteCarloRuns > 0. The cWithTolerance5_0(x) function provides a uniform distribution of ±5% initial and ±1% temperature. The cWithTolerance2_0(x) function provides a uniform distribution of ±2% initial and ±1% temperature. The rWithTolerance1_0(x) function provides a uniform distribution of ±1% initial and ±1% temperature. The rW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"
- note removed: ".control setplot const let numberOfMonteCarloRuns = 0 let areFiltersAdjusted = 1 let arePgasAdjusted = 1 let isAdcBufferAdjusted = 1 let rngSeed = 1 + rnd(2^32-2) let Rfilt1 = 4.3k let Rfilt2 = 68 let Rfilt3 = 54.9k let Rfilt4 = 4.3k let Cfilt1 = 4.7n let Cfilt2 = 360p let Rpga1 = 100 let Rpga2 = 390 let Rpga3 = 1.24k let Rpga4 = 2.49k let Rpga5 = 4.99k let Cpga1 = 100p let CpgaDecoupling1 = 4.7n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"
- note removed: ".tran 200n 500u 0"
- note removed: "To run a Monte-Carlo simulation, set numberOfMonteCarloRuns > 0. The cWithTolerance5_0(x) function provides a uniform distribution of ±5% initial and ±1% temperature. The cWithTolerance2_0(x) function provides a uniform distribution of ±2% initial and ±1% temperature. The rWithTolerance1_0(x) function provides a uniform distribution of ±1% initial and ±1% temperature. The rWithTolerance0_1(x) fun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"
- moved on the sheet: Cbypass1, L1, L2, RL1_1, RL1_2, Rvdd1, Rvref1, V1, V3

Commit message: Lots of faffing around trying to get ngspice to (reliably) converge for the MSF front-end, particularly around the Monte-Carlo simulations which seem to diverge for some values - it even appears as though some state is being held onto / corrupted between plots.  A good range of values has been tested and they agree nicely with each other, however.  Enough confidence exists to build it.  Also selected a new op-amp and removed the AZ431 voltage reference in favour of an op-amp solution, based on feedback from the simulations.  Noise and dynamic range estimations are satisfactory for this application, ADC and filter order.
Parts:
- removed Rvdd1: ${SIM.PARAMS}, restall-generic-resistors:nominal-0402-1005, symbol restall-generic-resistors:resistor
- added Cbypass7: 22u, restall-generic-capacitors:unpolarised-nominal-0805-2012, symbol restall-generic-capacitors:capacitor-unpolarised
- added Radc10, Radc9, Rmsf2, Rsim_1, Rsim_2, Rsim_3, Rsim_4, Rsim_5, Rsim_6, Rsim_7: ${SIM.PARAMS}, restall-generic-resistors:nominal-0402-1005, symbol restall-generic-resistors:resistor
- added V4: AM, symbol Simulation_SPICE:VSIN
- Cref1: value ${SIM.PARAMS} -> 4.7u
- U1, U2, U3, U4, U5, U6, U7: value MCP6486 -> MCP6496
- Vsimforce1: value 1.25 -> 1.8
Connections:
- net GND: now also Cref1.2, Cbypass7.2, Radc10.1, V4.2; no longer Cref1.1
- net V_{dd+3.6V}: now also V3.1
- net V_{out1}: now also Rsim_1.2; no longer U1.3
- net V_{out2}: now also Rsim_2.2; no longer U2.3
- net V_{out3}: now also Rsim_5.2; no longer U3.3
- net V_{out4}: now also Rsim_4.2; no longer U4.3
- net Vref_{+2.5V}: now also Radc9.2; no longer Rref1.2
- net V_{olin+}: now reaches Uol1.1 (+), Volac1.1
- net at Radc2.2, Radc4.2, Radc6.2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: now also Rsim_7.2; no longer U6.3
- net at Radc3.2, Radc5.2, Radc7.1: now also Rsim_6.2; no longer U5.3
- net V_{in+7}: now reaches Rref1.1, Rref2.2, U7.1 (+)
- net V_{in+7}: now also Cref1.1; no longer Cref1.2
- net V_{in-7}: now reaches Cref2.1, Rref3.1, U7.2 (-)
- net at Cref2.2, Rref3.2, Rref4.1: now also Rsim_3.2; no longer U7.3
- net V_{in-4}: now reaches Cfilt2_2.2, Rfilt2_4.1, U4.2 (-)
- net V_{in-2}: now reaches Cfilt1_2.2, Rfilt1_4.1, U2.2 (-)
- net V_{msfsim}: now reaches L2.1 (P1), Rmsf1.1
- net V_{msfsim}: now also Rmsf2.1
- net V_{olin-}: now reaches Col1.1, Rol1.1, Uol1.2 (-)
- net Vref_{+1.25V} renamed Vref_{+1.8V}
- net Vref_{+1.8V}: now also Cbypass7.1; no longer Cbypass4.1, U6.1 (+)
- new net: Rsim_2.1, U2.3
- new net: Rsim_7.1, U6.3
- new net: Rsim_3.1, U7.3
- new net: Rsim_4.1, U4.3
- new net: Rsim_6.1, U5.3
- new net: Cbypass4.1, Radc10.2, Radc9.1, U6.1 (+)
- new net: Rsim_1.1, U1.3
- new net: Rsim_5.1, U3.3
- new net V_{amsim}: Rmsf2.2, V4.1
- new net Vdd_{+3.6V}: Rref1.2
Other:
- note added: "!!! NOTE !!! CURRENTLY EXCLUDED FROM SIMULATION TO PREVENT RANDOM CONVERGENCE ISSUES DURING MONTE-CARLO ANALYSES ! THIS AOP SIM DOESN'T CONVERGE WITH THE MCP6496 MODEL ! The MCP6486 works, so that is used instead (lower bandwidth model so the headroom requirement should easily be met)."
- note added: "!!! NOTE !!! If convergence failure close to start of simulation, try playing with the 'msfDelay' parameter for the AM source."
- note added: "!!! NOTE !!! The TMUX1511 model has some .nodesets in it. It may be necessary to (un)comment these if there are convergence issues."
- note added: "*nodeset v(/Volin+)=1.8 *nodeset v(/Volin-)=1.8 *nodeset v(/Volvdd1)=3.6 *nodeset v(/Volac1)=1.8"
- note added: "*tran 10n 5m 0"
- note added: ".control setplot const let isNoiseAnalysis = 0 let numberOfMonteCarloRuns = 10 let areFiltersAdjusted = 1 let arePgasAdjusted = 1 let isAdcBufferAdjusted = 1 let rngSeed = 1 + rnd(2^32-2) let Rfilt1 = 4.12k let Rfilt2 = 64.9 let Rfilt3 = 49.9k let Rfilt4 = 10m let Cfilt1 = 4.7n let Cfilt2 = 470p let Rpga1_1 = 47 let Rpga2_1 = 100 let Rpga2 = 390 let Rpga3 = 1.24k let Rpga4 = 2.49k let Rpga5 = 4.9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"
- note added: ".nodeset v(/Vdd+3.6V)=3.6 .nodeset v(/Vmsfsim)=0 .nodeset v(/Vmsf)=1.8 .nodeset v(/Vref+2.5V)=2.5 .nodeset v(/Vref+1.8V)=1.8 .nodeset v(/Vin+1)=1.8 .nodeset v(/Vin-1)=1.8 .nodeset v(/Vout1)=1.8 .nodeset v(/Vin-2)=1.8 .nodeset v(/Vout2)=1.8 .nodeset v(/Vin+3)=1.8 .nodeset v(/Vin-3)=1.8 .nodeset v(/Vout3)=1.8 .nodeset v(/Vin-4)=1.8 .nodeset v(/Vout4)=1.8 .nodeset v(/Vin+7)=1.8 .nodeset v(/Vin-7)=1.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"
- note added: ".op"
- note added: ".options Rshunt=10G gmin=0.1p"
- note added: ".param adcGainR=2.49k .param adcFeedbackR=2.49k .param isMsfAmplitudeModulated=0 .param msfMagnitudeV=1.35 .param msfDelay=3u"
- note added: "Cross-over distortion will occur around VDD-0.9V for the non-inverting configurations. This shouldn't be a problem with a VDD/2 reference since the signals of interest will mainly be low-level. Even if they aren't then the distortion will be harmonics (120kHz, 180kHz, etc.) The 180kHz is the worst in terms of aliasing but the filters will attenuate > 80dB. The application is essentially a tone de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"
- note added: "For 118Hz bandwidth: Noise for gain at max/max (~85.5dB; ~89dB anti-aliasing) and 14-bit anti-aliasing filtering: 60kHz - 241.5μV/Hz^{-1} / 3.3mV_{rms}, about 22 lost codes 180kHz - 306nV/Hz^{-1} / 4.2μV_{rms}, noise << LSb Noise for gain at max/min (~47.7dB; ~88.2dB anti-aliasing) and 14-bit anti-aliasing filtering: 60kHz - 3.26μV/Hz^{-1} / 44.4μV_{rms}, noise << LSb Noise for gain at min/max (~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"
- note added: "For V2 transient simulation, set V=130μV_{pp} with maximum gain or V=1.35V_{pp} with minimum gain. Both result in about 2.34V_{pp} at the ADC, around 93% of full scale. This is a result of the opamp hitting the lower-rail limit of swing, plus the RC anti-aliasing filter loss."
- note added: "Full-scale (~2.5V_{p-p} at the ADC) is ~130μV_{p-p} on maximum gain. About 7% ADC headroom, which is the opamp lower-rail limit plus loss of the ADC RC anti-aliasing filter."
- note added: "Monte-Carlo on 100 runs for differential ADC voltage with maximum PGA gain: +81.5dB to +79.5dB @ 60kHz -16.9 to -18.5dB @ 180kHz About 15 bits Monte-Carlo on 100 runs for differential ADC voltage with minimum PGA gain: +10.5dB to +7.6dB @ 60kHz -74.6dB to -75.5dB @ 180kHz About 13 bits !!! NOTE !!! Figures above are inaccurate as large Monte-Carlo runs fail with convergence issues in some simulat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"
- note added: "Noise at the ADC is about 1.4μV/Hz^{-1} at 60kHz for minimum gain. Assuming a DFT with 1024 bins and an ADC sampling at 240kHz (about 5ms latency), each bin has a bandwidth of 235Hz. Using a filter shape factor of 1.57 we get: 1.4μV/Hz^{-1} * sqrt(235 * 1.57) = 26.9μV_{rms} That equates to about three quarters of an LSb for 16-bit sampling, but the anti-aliasing filter can only reject the first a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"
- note added: "Open Loop Gain Measurement Rule of thumb (Op-Amps for Everyone, p461) - active filters need +40dB A_{o} headroom above filter response peak. The MCP6489 model does not vary A_{o} over V_{dd}, etc. so ensure an additional -6dB headroom to allow PVT variation."
- note added: "Virtual Ground Voltage Reference"
- note removed: "*noise v(/Vadc+, /Vadc-) V2 lin 10k 1 10Meg"
- note removed: "*tran 200n 500u 0"
- note removed: ".control setplot const let isNoiseAnalysis = 1 let numberOfMonteCarloRuns = 0 let areFiltersAdjusted = 1 let arePgasAdjusted = 1 let isAdcBufferAdjusted = 1 let rngSeed = 1 + rnd(2^32-2) let Rfilt1 = 4.3k let Rfilt2 = 68 let Rfilt3 = 54.9k let Rfilt4 = 4.3k let Cfilt1 = 4.7n let Cfilt2 = 360p let Rpga1 = 100 let Rpga2 = 390 let Rpga3 = 1.24k let Rpga4 = 2.49k let Rpga5 = 4.99k let Cpga1 = 100p le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"
- note removed: ".nodeset v(/Vref+1.25V)=1.25 .nodeset v(/Vin+1)=1.25 .nodeset v(/Vin+3)=1.25 .nodeset v(/Vin+5)=1.25 .nodeset v(/Vin-5)=1.25 .nodeset v(/Vin-6)=1.25"
- note removed: ".options Rshunt=10G Cshunt=0.1p gmin=0.1p reltol=0.01"
- note removed: ".param adcGainR=2.49k .param adcFeedbackR=2.49k"
- note removed: "ADC Common-Mode Voltage Reference"
- note removed: "For V2 transient simulation, set V=410u with maximum gain or V=1.55V with minimum gain"
- note removed: "Full-scale (~2.5V_{p-p} at the ADC) is ~410μV_{p-p} on maximum gain"
- note removed: "Monte-Carlo on 100 runs for differential ADC voltage with maximum PGA gain: +81.5dB to +79.5dB @ 60kHz -16.9 to -18.5dB @ 180kHz About 15 bits Monte-Carlo on 100 runs for differential ADC voltage with minimum PGA gain: +10.5dB to +7.6dB @ 60kHz -74.6dB to -75.5dB @ 180kHz About 13 bits"
- note removed: "Noise at the ADC is about 2.32μV/Hz^{-1} at 60kHz for minimum gain. Assuming a DFT with 1024 bins and an ADC sampling at 240kHz (about 5ms latency), each bin has a bandwidth of 235Hz. Using a filter shape factor of 1.57 we get: 2.32μV/Hz^{-1} * sqrt(235 * 1.57) = 44.6μV_{rms} That equates to just over half an LSb for 15-bit sampling. We can of course decrease the bin with at the expense of latenc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"
- note removed: "Open Loop Gain Measurement Rule of thumb (Op-Amps for Everyone, p461) - active filters need +40dB A_{o} headroom above filter response peak. The MCP6849 model does not vary A_{o} over V_{dd}, etc. so ensure an additional -6dB headroom to allow PVT variation."
- moved on the sheet: Cadc1, Radc7, Radc8, Rmsf1, Rvref1, V1, V2, V3
