File: sim/msf-front-end/msf-front-end.kicad_sch (KiCad schematic)
At the start: 94 parts, among them K1 TMUX1511, K2 TMUX1511, K3 TMUX1511, K4 TMUX1511, K5 TMUX1511, K6 TMUX1511, K7 TMUX1511, K8 TMUX1511, U1 MCP6496, U2 MCP6496, U3 MCP6496, U4 MCP6496, U5 MCP6496, U6 MCP6496, U7 MCP6496

Commit message: Re-running some simulations.  Plus fixed a capacitor model that was biased for 1.25V when really it ought to have been 1.8V based on the in-circuit voltage.
Parts:
- added Rvdd1: ${SIM.PARAMS}, restall-generic-resistors:nominal-0402-1005, symbol restall-generic-resistors:resistor
- added Vadcdiff1: ${SIM.PARAMS}, symbol Simulation_SPICE:VSIN
Connections:
- net GND: now also Vadcdiff1.2; no longer K1.A1, K2.A1, K3.A1, K4.A1, K5.A1, K6.A1, K7.A1, K8.A1
- net V_{dd+3.6V}: now also K1.A1, K2.A1, K3.A1, K4.A1, K5.A1, K6.A1, K7.A1, K8.A1, Rvdd1.1; no longer V3.1
- new net: Rvdd1.2, V3.1
- new net V_{adcdiff}: Vadcdiff1.1
Other:
- note added: "!!! NOTE !!! Rvref1 and Rvdd1 are sometimes required for convergence. Sometimes they prevent convergence. Tweak accordingly."
- note added: "*op"
- note added: ".ac lin 10k 1 10Meg"
- note added: ".control setplot const let isNoiseAnalysis = 0 let numberOfMonteCarloRuns = 0 let areFiltersAdjusted = 1 let arePgasAdjusted = 1 let isAdcBufferAdjusted = 1 let rngSeed = 1 + rnd(2^32-2) let Rfilt1 = 4.12k let Rfilt2 = 64.9 let Rfilt3 = 49.9k let Rfilt4 = 10m let Cfilt1 = 4.7n let Cfilt2 = 470p let Rpga1_1 = 47 let Rpga2_1 = 100 let Rpga2 = 390 let Rpga3 = 1.24k let Rpga4 = 2.49k let Rpga5 = 4.99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"
- note removed: "*ac lin 10k 1 10Meg"
- note removed: ".control setplot const let isNoiseAnalysis = 0 let numberOfMonteCarloRuns = 10 let areFiltersAdjusted = 1 let arePgasAdjusted = 1 let isAdcBufferAdjusted = 1 let rngSeed = 1 + rnd(2^32-2) let Rfilt1 = 4.12k let Rfilt2 = 64.9 let Rfilt3 = 49.9k let Rfilt4 = 10m let Cfilt1 = 4.7n let Cfilt2 = 470p let Rpga1_1 = 47 let Rpga2_1 = 100 let Rpga2 = 390 let Rpga3 = 1.24k let Rpga4 = 2.49k let Rpga5 = 4.9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"
- note removed: ".op"
