File: sim/msf-front-end/msf-front-end.kicad_sch (KiCad schematic)
At the start: 96 parts, among them K1 TMUX1511, K2 TMUX1511, K3 TMUX1511, K4 TMUX1511, K5 TMUX1511, K6 TMUX1511, K7 TMUX1511, K8 TMUX1511, U1 MCP6496, U2 MCP6496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

Commit message: Investigated the effect of some bypass networks on the op-amp outputs (PSRR).
Parts:
- added Cbypass10, Cbypass8, Cbypass9: 22u, restall-generic-capacitors:unpolarised-nominal-0805-2012, symbol restall-generic-capacitors:capacitor-unpolarised
- added Cbypass11, Cbypass12: 4.7u, restall-generic-capacitors:unpolarised-nominal-0402-1005, symbol restall-generic-capacitors:capacitor-unpolarised
Connections:
- net GND: now also Cbypass10.2, Cbypass11.2, Cbypass12.2, Cbypass8.2, Cbypass9.2
- net V_{dd+3.6V}: now also Cbypass10.1, Cbypass11.1, Cbypass12.1, Cbypass8.1, Cbypass9.1
Other:
- note added: "!!! NOTE !!! PSRR@60kHz in the MCP6496 model looks to be about -16dB as opposed to the -50dB from the datasheet (at 5.5V). That's a big difference, but it does appear to be modelled at least, which should give confidence that the bypass network is in the right ballpark."
- note added: "*ac lin 10k 1 10Meg"
- note added: ".options Rshunt=10G gmin=0.1p method=gear"
- note added: ".param adcGainR=2.49k .param adcFeedbackR=2.49k .param isMsfAmplitudeModulated=1 .param msfMagnitudeV=1.3 .param msfDelay=3u"
- note added: ".tran 100n 5m 0"
- note removed: "*tran 10n 5m 0"
- note removed: ".ac lin 10k 1 10Meg"
- note removed: ".options Rshunt=10G gmin=0.1p"
- note removed: ".param adcGainR=2.49k .param adcFeedbackR=2.49k .param isMsfAmplitudeModulated=0 .param msfMagnitudeV=1.35 .param msfDelay=3u"
- moved on the sheet: Cbypass5, Cbypass6, Cbypass7
