File: src/schematics/2-msf-receiver-trf.kicad_sch (KiCad schematic)
At the start: 33 parts, among them U203 MCP6499, U204 MCP6499, U206 TMUX1511RSV

Commit message: Further elaboration of the MSF front-end.
Parts:
- added C242, C243: 4.7μF, restall-generic-capacitors:unpolarised-nominal-0402-1005, symbol restall-generic-capacitors:capacitor-unpolarised
- added U207: TMUX1511RSV, restall-manufacturer-ti:UQFN16-1.8x2.6mm-0.4mm, symbol restall-manufacturer-ti:TMUX1511RSV
- renumbered C46 to C232, C49 to C233, C47 to C234, C40 to C235, C44 to C236, C43 to C237, C50 to C238, C48 to C239, C41 to C240, C45 to C241, R37 to R225, R51 to R226, R43 to R227, R44 to R228, R45 to R229, R46 to R230, R38 to R231, R41 to R232, R33 to R233, R35 to R234, R40 to R235, R52 to R236, R47 to R237, R48 to R238, R49 to R239, R50 to R240, R39 to R241, R42 to R242, R34 to R243, R36 to R244
Connections:
- net FB0: now also U206.10, U207.10
- net FB1: now also U206.6, U206.9, U207.6, U207.9
- net FB2: now also U206.3, U206.5, U207.3, U207.5
- net FB3: now also U206.14, U206.2, U207.14, U207.2
- net FB4: now also U206.13, U207.13
- net GND: now also U206.12 (V_{SS}), U206.7 (V_{SS}), U206.8 (V_{SS}), C242.2, C243.2, U207.12 (V_{SS}), U207.7 (V_{SS}), U207.8 (V_{SS})
- net MSF_VDD_{+3.6V}: now also U206.16 (V_{DD}), C242.1, C243.1, U207.16 (V_{DD})
- net SW_EN3: now reaches U206.15
- net SW_EN3: now also U207.15
- net SW_EN0: now reaches U206.11
- net SW_EN0: now also U207.11
- net SW_EN1: now reaches U206.4
- net SW_EN1: now also U207.4
- net SW_EN2: now reaches U206.1
- net SW_EN2: now also U207.1
Other:
- note added: "MFB Bandpass, f_{0}≃60kHz, Q≃8, K≃-1.1 Split R233 / R234 provides opportunity for a Deliyannis topology if desired."
- note added: "MFB Bandpass, f_{0}≃60kHz, Q≃8, K≃-1.1 Split R243 / R244 provides opportunity for a Deliyannis topology if desired."
- note removed: "MFB Bandpass, f_{0}≃60kHz, Q≃8, K≃-1.1 Split R2xx / R2yy provides opportunity for a Deliyannis topology if desired."
- note removed: "TODO: ADD SWITCHES"
- note removed: "TODO: BYPASS CAPS"
- note removed: "TODO: PAPER AND PENCIL - FIGURE OUT THE BEST ORIENTATION FOR THE SWITCHES"
- moved on the sheet: U206A, U206B, U206C, U206D, U206E

Commit message: Typo.
Other:
- note added: "Tuned RF Section 1"
- note added: "Tuned RF Section 2"
- note removed: "Tuned RF Secion 1"
- note removed: "Tuned RF Secion 2"
Changed lines of the file:
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@@
     (effects (font (size 1.27 1.27)) (justify left bottom))
   )
-  (text "Tuned RF Secion 2" (at 302.26 37.338 0)
+  (text "Tuned RF Section 2" (at 302.26 37.338 0)
     (effects (font (size 2.54 2.54)) (justify left bottom))
   )
@@
     (effects (font (size 1.27 1.27)) (justify left bottom))
   )
-  (text "Tuned RF Secion 1" (at 104.14 37.338 0)
+  (text "Tuned RF Section 1" (at 104.14 37.338 0)
     (effects (font (size 2.54 2.54)) (justify left bottom))
   )

Commit message: Finished drawing up the audio output schematic.  The speaker selection is still to do.
Changed lines of the file:
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@@
   (symbol (lib_id "restall-generic-capacitors:capacitor-unpolarised") (at 261.62 114.3 0) (unit 1)
     (in_bom yes) (on_board yes) (dnp no)
-    (property "Reference" "C238" (at 264.16 113.538 0)
-      (effects (font (size 1.27 1.27)) (justify left))
-    )
-    (property "Value" "4.7μF" (at 264.16 115.57 0)
+    (property "Reference" "C238" (at 264.16 113.284 0)
+      (effects (font (size 1.27 1.27)) (justify left))
+    )
+    (property "Value" "4.7μF" (at 264.16 115.316 0)
       (effects (font (size 1.27 1.27)) (justify left))
     )
@@
   (symbol (lib_id "restall-generic-capacitors:capacitor-unpolarised") (at 38.1 149.86 0) (unit 1)
     (in_bom yes) (on_board yes) (dnp no)
-    (property "Reference" "C242" (at 40.64 149.098 0)
-      (effects (font (size 1.27 1.27)) (justify left))
-    )
-    (property "Value" "4.7μF" (at 40.64 151.13 0)
+    (property "Reference" "C242" (at 40.64 148.844 0)
+      (effects (font (size 1.27 1.27)) (justify left))
+    )
+    (property "Value" "4.7μF" (at 40.64 150.876 0)
       (effects (font (size 1.27 1.27)) (justify left))
     )
@@
   (symbol (lib_id "restall-generic-capacitors:capacitor-unpolarised") (at 243.84 149.86 0) (unit 1)
     (in_bom yes) (on_board yes) (dnp no)
-    (property "Reference" "C243" (at 246.38 149.098 0)
-      (effects (font (size 1.27 1.27)) (justify left))
-    )
-    (property "Value" "4.7μF" (at 246.38 151.13 0)
+    (property "Reference" "C243" (at 246.38 148.844 0)
+      (effects (font (size 1.27 1.27)) (justify left))
+    )
+    (property "Value" "4.7μF" (at 246.38 150.876 0)
       (effects (font (size 1.27 1.27)) (justify left))
     )
@@
   (symbol (lib_id "restall-generic-capacitors:capacitor-unpolarised") (at 63.5 114.3 0) (unit 1)
     (in_bom yes) (on_board yes) (dnp no)
-    (property "Reference" "C233" (at 66.04 113.538 0)
-      (effects (font (size 1.27 1.27)) (justify left))
-    )
-    (property "Value" "4.7μF" (at 66.04 115.57 0)
+    (property "Reference" "C233" (at 66.04 113.284 0)
+      (effects (font (size 1.27 1.27)) (justify left))
+    )
+    (property "Value" "4.7μF" (at 66.04 115.316 0)
       (effects (font (size 1.27 1.27)) (justify left))
     )
@@
   (symbol (lib_id "restall-generic-capacitors:capacitor-unpolarised") (at 35.56 83.82 0) (unit 1)
     (in_bom yes) (on_board yes) (dnp no)
-    (property "Reference" "C232" (at 38.1 83.058 0)
-      (effects (font (size 1.27 1.27)) (justify left))
-    )
-    (property "Value" "4.7μF" (at 38.1 85.09 0)
-      (effects (font (size 1.27 1.27)) (justify left))
-    )
+    (property "Reference" "C232" (at 38.1 82.804 0)
+      (effects (font (size 1.27 1.27)) (justify left))
+    )
+    (property "Value" "4.7μF" (at 38.1 84.836 0)
+      (effects (font (size 1.27 1.27)) (justify left))
+    )

Commit message: Added another bypass capacitor.
Parts:
- renumbered C232 to C233, C233 to C234, C234 to C235, C235 to C236, C236 to C237, C237 to C238, C238 to C239, C239 to C240, C240 to C241, C241 to C242, C242 to C243, C243 to C244
Changed lines of the file:
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@@
   (symbol (lib_id "restall-generic-capacitors:capacitor-unpolarised") (at 90.17 86.36 90) (unit 1)
     (in_bom no) (on_board yes) (dnp no)
-    (property "Reference" "C234" (at 88.138 76.708 90)
+    (property "Reference" "C235" (at 88.138 76.708 90)
       (effects (font (size 1.27 1.27)) (justify right))
     )
@@
       (project "msf-owl-clock"
         (path "/56d623d3-22db-4d43-a9d9-e6bb4bb68946/ce863d79-d266-4984-b56b-ca957df41c84/4fbb3fbf-2c3d-43d2-97c2-d56faba30b72"
-          (reference "C234") (unit 1)
+          (reference "C235") (unit 1)
         )
       )
@@
   (symbol (lib_id "restall-generic-capacitors:capacitor-unpolarised") (at 245.11 68.58 270) (unit 1)
     (in_bom yes) (on_board yes) (dnp no)
-    (property "Reference" "C237" (at 242.57 56.642 90)
+    (property "Reference" "C238" (at 242.57 56.642 90)
       (effects (font (size 1.27 1.27)) (justify left))
     )
@@
       (project "msf-owl-clock"
         (path "/56d623d3-22db-4d43-a9d9-e6bb4bb68946/ce863d79-d266-4984-b56b-ca957df41c84/4fbb3fbf-2c3d-43d2-97c2-d56faba30b72"
-          (reference "C237") (unit 1)
+          (reference "C238") (unit 1)
         )
       )
@@
   (symbol (lib_id "restall-generic-capacitors:capacitor-unpolarised") (at 137.16 57.15 180) (unit 1)
     (in_bom yes) (on_board yes) (dnp no)
-    (property "Reference" "C235" (at 139.7 53.086 0)
+    (property "Reference" "C236" (at 139.7 53.086 0)
       (effects (font (size 1.27 1.27)) (justify right))
     )
@@
       (project "msf-owl-clock"
         (path "/56d623d3-22db-4d43-a9d9-e6bb4bb68946/ce863d79-d266-4984-b56b-ca957df41c84/4fbb3fbf-2c3d-43d2-97c2-d56faba30b72"
-          (reference "C235") (unit 1)
+          (reference "C236") (unit 1)
         )
       )
@@
   (symbol (lib_id "restall-generic-capacitors:capacitor-unpolarised") (at 261.62 114.3 0) (unit 1)
     (in_bom yes) (on_board yes) (dnp no)
-    (property "Reference" "C238" (at 264.16 113.284 0)
+    (property "Reference" "C239" (at 264.16 113.284 0)
       (effects (font (size 1.27 1.27)) (justify left))
     )
@@
       (project "msf-owl-clock"
         (path "/56d623d3-22db-4d43-a9d9-e6bb4bb68946/ce863d79-d266-4984-b56b-ca957df41c84/4fbb3fbf-2c3d-43d2-97c2-d56faba30b72"
-          (reference "C238") (unit 1)
+          (reference "C239") (unit 1)
         )
       )
@@
   (symbol (lib_id "restall-generic-capacitors:capacitor-unpolarised") (at 344.17 73.66 90) (unit 1)
     (in_bom yes) (on_board yes) (dnp no)
-    (property "Reference" "C241" (at 342.138 63.754 90)
+    (property "Reference" "C242" (at 342.138 63.754 90)
       (effects (font (size 1.27 1.27)) (justify right))
     )
@@
       (project "msf-owl-clock"
         (path "/56d623d3-22db-4d43-a9d9-e6bb4bb68946/ce863d79-d266-4984-b56b-ca957df41c84/4fbb3fbf-2c3d-43d2-97c2-d56faba30b72"
-          (reference "C241") (unit 1)
+          (reference "C242") (unit 1)
         )
       )
@@
   (symbol (lib_id "restall-generic-capacitors:capacitor-unpolarised") (at 38.1 149.86 0) (unit 1)
     (in_bom yes) (on_board yes) (dnp no)
-    (property "Reference" "C242" (at 40.64 148.844 0)
+    (property "Reference" "C243" (at 40.64 148.844 0)
       (effects (font (size 1.27 1.27)) (justify left))
     )
@@
       (project "msf-owl-clock"
         (path "/56d623d3-22db-4d43-a9d9-e6bb4bb68946/ce863d79-d266-4984-b56b-ca957df41c84/4fbb3fbf-2c3d-43d2-97c2-d56faba30b72"
-          (reference "C242") (unit 1)
+          (reference "C243") (unit 1)
         )
       )
@@
   (symbol (lib_id "restall-generic-capacitors:capacitor-unpolarised") (at 288.29 86.36 90) (unit 1)
     (in_bom no) (on_board yes) (dnp no)
-    (property "Reference" "C239" (at 286.258 76.708 90)
+    (property "Reference" "C240" (at 286.258 76.708 90)
       (effects (font (size 1.27 1.27)) (justify right))
     )
@@
       (project "msf-owl-clock"
         (path "/56d623d3-22db-4d43-a9d9-e6bb4bb68946/ce863d79-d266-4984-b56b-ca957df41c84/4fbb3fbf-2c3d-43d2-97c2-d56faba30b72"
-          (reference "C239") (unit 1)
+          (reference "C240") (unit 1)
         )
       )
@@
   (symbol (lib_id "restall-generic-capacitors:capacitor-unpolarised") (at 146.05 73.66 90) (unit 1)
     (in_bom yes) (on_board yes) (dnp no)
-    (property "Reference" "C236" (at 144.018 63.754 90)
+    (property "Reference" "C237" (at 144.018 63.754 90)
       (effects (font (size 1.27 1.27)) (justify right))
     )
@@
       (project "msf-owl-clock"
         (path "/56d623d3-22db-4d43-a9d9-e6bb4bb68946/ce863d79-d266-4984-b56b-ca957df41c84/4fbb3fbf-2c3d-43d2-97c2-d56faba30b72"
-          (reference "C236") (unit 1)
+          (reference "C237") (unit 1)
         )
       )
@@
   (symbol (lib_id "restall-generic-capacitors:capacitor-unpolarised") (at 243.84 149.86 0) (unit 1)
     (in_bom yes) (on_board yes) (dnp no)
-    (property "Reference" "C243" (at 246.38 148.844 0)
+    (property "Reference" "C244" (at 246.38 148.844 0)
       (effects (font (size 1.27 1.27)) (justify left))
     )
@@
       (project "msf-owl-clock"
         (path "/56d623d3-22db-4d43-a9d9-e6bb4bb68946/ce863d79-d266-4984-b56b-ca957df41c84/4fbb3fbf-2c3d-43d2-97c2-d56faba30b72"
-          (reference "C243") (unit 1)
+          (reference "C244") (unit 1)
         )
       )
@@
   (symbol (lib_id "restall-generic-capacitors:capacitor-unpolarised") (at 63.5 114.3 0) (unit 1)
     (in_bom yes) (on_board yes) (dnp no)
-    (property "Reference" "C233" (at 66.04 113.284 0)
+    (property "Reference" "C234" (at 66.04 113.284 0)
       (effects (font (size 1.27 1.27)) (justify left))
     )
@@
       (project "msf-owl-clock"
         (path "/56d623d3-22db-4d43-a9d9-e6bb4bb68946/ce863d79-d266-4984-b56b-ca957df41c84/4fbb3fbf-2c3d-43d2-97c2-d56faba30b72"
-          (reference "C233") (unit 1)
+          (reference "C234") (unit 1)
         )
       )
@@
   (symbol (lib_id "restall-generic-capacitors:capacitor-unpolarised") (at 35.56 83.82 0) (unit 1)
     (in_bom yes) (on_board yes) (dnp no)
-    (property "Reference" "C232" (at 38.1 82.804 0)
+    (property "Reference" "C233" (at 38.1 82.804 0)
       (effects (font (size 1.27 1.27)) (justify left))
     )
@@
       (project "msf-owl-clock"
         (path "/56d623d3-22db-4d43-a9d9-e6bb4bb68946/ce863d79-d266-4984-b56b-ca957df41c84/4fbb3fbf-2c3d-43d2-97c2-d56faba30b72"
-          (reference "C232") (unit 1)
+          (reference "C233") (unit 1)
         )
       )
@@
   (symbol (lib_id "restall-generic-capacitors:capacitor-unpolarised") (at 335.28 57.15 180) (unit 1)
     (in_bom yes) (on_board yes) (dnp no)
-    (property "Reference" "C240" (at 337.82 53.086 0)
+    (property "Reference" "C241" (at 337.82 53.086 0)
       (effects (font (size 1.27 1.27)) (justify right))
     )
@@
       (project "msf-owl-clock"
         (path "/56d623d3-22db-4d43-a9d9-e6bb4bb68946/ce863d79-d266-4984-b56b-ca957df41c84/4fbb3fbf-2c3d-43d2-97c2-d56faba30b72"
-          (reference "C240") (unit 1)
-        )
-      )
+          (reference "C241") (unit 1)
+        )
+      )

Commit message: Various tidy-ups and checks, mainly around the bypass capacitors.  Added a load of test points.
Parts:
- added TP207, TP208, TP209: ~, restall-generic-test:testpoint-SP3050A-with-short-gnd, symbol restall-generic-test:testpoint-probe-with-gnd
Connections:
- net GND: now also TP207.2 (GND), TP208.2 (GND), TP209.2 (GND)
- net MSF_RCV_TRF: now also TP209.1
- net at C238.1, R235.1, U204.5 (+): now also TP208.1
- net at R225.2, U203.3 (+): now also TP207.1
Changed lines of the file:
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@@
   (junction (at 283.21 99.06) (diameter 0) (color 0 0 0 0)
   )
+  (junction (at 71.12 68.58) (diameter 0) (color 0 0 0 0)
+  )
   (junction (at 243.84 144.78) (diameter 0) (color 0 0 0 0)
   )
@@
   (junction (at 353.06 50.8) (diameter 0) (color 0 0 0 0)
   )
+  (junction (at 269.24 68.58) (diameter 0) (color 0 0 0 0)
+  )
   (junction (at 293.37 99.06) (diameter 0) (color 0 0 0 0)
   )
+  (junction (at 388.62 78.74) (diameter 0) (color 0 0 0 0)
+  )
   (junction (at 105.41 99.06) (diameter 0) (color 0 0 0 0)
   )
@@
     (stroke (width 0) (type default))
   )
-  (wire (pts (xy 251.46 68.58) (xy 271.78 68.58))
+  (wire (pts (xy 251.46 68.58) (xy 269.24 68.58))
     (stroke (width 0) (type default))
   )
@@
     (stroke (width 0) (type default))
   )
+  (wire (pts (xy 388.62 78.74) (xy 391.16 78.74))
+    (stroke (width 0) (type default))
+  )
   (wire (pts (xy 313.69 99.06) (xy 313.69 104.14))
     (stroke (width 0) (type default))
@@
     (stroke (width 0) (type default))
   )
+  (wire (pts (xy 71.12 62.23) (xy 71.12 68.58))
+    (stroke (width 0) (type default))
+  )
   (wire (pts (xy 261.62 99.06) (xy 261.62 100.33))
     (stroke (width 0) (type default))
@@
     (stroke (width 0) (type default))
   )
-  (wire (pts (xy 386.08 78.74) (xy 391.16 78.74))
+  (wire (pts (xy 386.08 78.74) (xy 388.62 78.74))
     (stroke (width 0) (type default))
   )
@@
     (stroke (width 0) (type default))
   )
+  (wire (pts (xy 71.12 68.58) (xy 73.66 68.58))
+    (stroke (width 0) (type default))
+  )
   (wire (pts (xy 85.09 99.06) (xy 83.82 99.06))
     (stroke (width 0) (type default))
@@
     (stroke (width 0) (type default))
   )
-  (wire (pts (xy 45.72 68.58) (xy 73.66 68.58))
+  (wire (pts (xy 45.72 68.58) (xy 71.12 68.58))
     (stroke (width 0) (type default))
   )
@@
     (stroke (width 0) (type default))
   )
+  (wire (pts (xy 269.24 62.23) (xy 269.24 68.58))
+    (stroke (width 0) (type default))
+  )
   (wire (pts (xy 353.06 50.8) (xy 386.08 50.8))
     (stroke (width 0) (type default))
@@
     (stroke (width 0) (type default))
   )
+  (wire (pts (xy 388.62 86.36) (xy 389.89 86.36))
+    (stroke (width 0) (type default))
+  )
   (wire (pts (xy 35.56 78.74) (xy 35.56 80.01))
     (stroke (width 0) (type default))
@@
     (stroke (width 0) (type default))
   )
+  (wire (pts (xy 388.62 78.74) (xy 388.62 86.36))
+    (stroke (width 0) (type default))
+  )
   (wire (pts (xy 261.62 99.06) (xy 273.05 99.06))
     (stroke (width 0) (type default))
@@
     (stroke (width 0) (type default))
   )
+  (wire (pts (xy 269.24 68.58) (xy 271.78 68.58))
+    (stroke (width 0) (type default))
+  )
   (bus (pts (xy 107.95 106.68) (xy 118.11 106.68))
     (stroke (width 0) (type default))
@@
     )
   )
+  (symbol (lib_id "restall-generic-power:GND") (at 68.072 62.23 0) (unit 1)
+    (in_bom yes) (on_board yes) (dnp no) (fields_autoplaced)
+    (property "Reference" "#PWR0273" (at 68.072 68.58 0)
+      (effects (font (size 1.27 1.27)) hide)
+    )
+    (property "Value" "GND" (at 68.072 66.3631 0)
+      (effects (font (size 1.27 1.27)))
+    )
+    (property "Footprint" "" (at 68.072 62.23 0)
+      (effects (font (size 1.27 1.27)) hide)
+    )
+    (property "Datasheet" "" (at 68.072 62.23 0)
+      (effects (font (size 1.27 1.27)) hide)
+    )
+    (pin "1")
+    (instances
+      (project "msf-owl-clock"
+        (path "/56d623d3-22db-4d43-a9d9-e6bb4bb68946/ce863d79-d266-4984-b56b-ca957df41c84/4fbb3fbf-2c3d-43d2-97c2-d56faba30b72"
+          (reference "#PWR0273") (unit 1)
+        )
+      )
+    )
+  )
   (symbol (lib_id "restall-generic-capacitors:capacitor-unpolarised") (at 245.11 68.58 270) (unit 1)
     (in_bom yes) (on_board yes) (dnp no)
@@
     )
   )
+  (symbol (lib_id "restall-generic-test:testpoint-probe-with-gnd") (at 71.12 62.23 0) (mirror y) (unit 1)
+    (in_bom no) (on_board yes) (dnp no)
+    (property "Reference" "TP207" (at 61.468 59.69 0)
+      (effects (font (size 1.27 1.27)) (justify right))
+    )
+    (property "Value" "~" (at 69.469 58.166 0)
+      (effects (font (size 1.27 1.27)) (justify right) hide)
+    )
+    (property "Footprint" "restall-generic-test:testpoint-SP3050A-with-short-gnd" (at 66.04 62.23 0)
+      (effects (font (size 1.27 1.27)) (justify right) hide)
+    )
+    (property "Datasheet" "~" (at 66.04 62.23 0)
+      (effects (font (size 1.27 1.27)) (justify right) hide)
+    )
+    (pin "2")
+    (pin "1")
+    (instances
+      (project "msf-owl-clock"
+        (path "/56d623d3-22db-4d43-a9d9-e6bb4bb68946/ce863d79-d266-4984-b56b-ca957df41c84/4fbb3fbf-2c3d-43d2-97c2-d56faba30b72"
+          (reference "TP207") (unit 1)
+        )
+      )
+    )
+  )
   (symbol (lib_id "restall-generic-resistors:resistor") (at 123.19 73.66 90) (unit 1)
     (in_bom yes) (on_board yes) (dnp no)
@@
     )
   )
+  (symbol (lib_id "restall-generic-power:GND") (at 266.192 62.23 0) (unit 1)
+    (in_bom yes) (on_board yes) (dnp no) (fields_autoplaced)
+    (property "Reference" "#PWR0274" (at 266.192 68.58 0)
+      (effects (font (size 1.27 1.27)) hide)
+    )
+    (property "Value" "GND" (at 266.192 66.3631 0)
+      (effects (font (size 1.27 1.27)))
+    )
+    (property "Footprint" "" (at 266.192 62.23 0)
+      (effects (font (size 1.27 1.27)) hide)
+    )
+    (property "Datasheet" "" (at 266.192 62.23 0)
+      (effects (font (size 1.27 1.27)) hide)
+    )
+    (pin "1")
+    (instances
+      (project "msf-owl-clock"
+        (path "/56d623d3-22db-4d43-a9d9-e6bb4bb68946/ce863d79-d266-4984-b56b-ca957df41c84/4fbb3fbf-2c3d-43d2-97c2-d56faba30b72"
+          (reference "#PWR0274") (unit 1)
+        )
+      )
+    )
+  )
   (symbol (lib_id "restall-manufacturer-microchip:MCP6499?-?-S?") (at 82.55 73.66 0) (unit 1)
     (in_bom yes) (on_board yes) (dnp no)
@@
     )
   )
+  (symbol (lib_id "restall-generic-test:testpoint-probe-with-gnd") (at 269.24 62.23 0) (mirror y) (unit 1)
+    (in_bom no) (on_board yes) (dnp no)
+    (property "Reference" "TP208" (at 259.588 59.69 0)
+      (effects (font (size 1.27 1.27)) (justify right))
+    )
+    (property "Value" "~" (at 267.589 58.166 0)
+      (effects (font (size 1.27 1.27)) (justify right) hide)
+    )
+    (property "Footprint" "restall-generic-test:testpoint-SP3050A-with-short-gnd" (at 264.16 62.23 0)
+      (effects (font (size 1.27 1.27)) (justify right) hide)
+    )
+    (property "Datasheet" "~" (at 264.16 62.23 0)
+      (effects (font (size 1.27 1.27)) (justify right) hide)
+    )
+    (pin "2")
+    (pin "1")
+    (instances
+      (project "msf-owl-clock"
+        (path "/56d623d3-22db-4d43-a9d9-e6bb4bb68946/ce863d79-d266-4984-b56b-ca957df41c84/4fbb3fbf-2c3d-43d2-97c2-d56faba30b72"
+          (reference "TP208") (unit 1)
+        )
+      )
+    )
+  )
   (symbol (lib_id "restall-generic-power:GND") (at 261.62 118.11 0) (unit 1)
     (in_bom yes) (on_board yes) (dnp no) (fields_autoplaced)
@@
     )
   )
+  (symbol (lib_id "restall-generic-power:GND") (at 392.938 86.36 0) (unit 1)
+    (in_bom yes) (on_board yes) (dnp no) (fields_autoplaced)
+    (property "Reference" "#PWR0275" (at 392.938 92.71 0)
+      (effects (font (size 1.27 1.27)) hide)
+    )
+    (property "Value" "GND" (at 392.938 90.4931 0)
+      (effects (font (size 1.27 1.27)))
+    )
+    (property "Footprint" "" (at 392.938 86.36 0)
+      (effects (font (size 1.27 1.27)) hide)
+    )
+    (property "Datasheet" "" (at 392.938 86.36 0)
+      (effects (font (size 1.27 1.27)) hide)
+    )
+    (pin "1")
+    (instances
+      (project "msf-owl-clock"
+        (path "/56d623d3-22db-4d43-a9d9-e6bb4bb68946/ce863d79-d266-4984-b56b-ca957df41c84/4fbb3fbf-2c3d-43d2-97c2-d56faba30b72"
+          (reference "#PWR0275") (unit 1)
+        )
+      )
+    )
+  )
   (symbol (lib_id "restall-generic-resistors:resistor") (at 353.06 57.15 0) (unit 1)
     (in_bom yes) (on_board yes) (dnp no)
@@
         )
       )
+    )
+  )
+  (symbol (lib_id "restall-generic-test:testpoint-probe-with-gnd") (at 389.89 86.36 0) (unit 1)
+    (in_bom no) (on_board yes) (dnp no)
+    (property "Reference" "TP209" (at 399.542 83.82 0)
+      (effects (font (size 1.27 1.27)) (justify right))
+    )
+    (property "Value" "~" (at 391.541 82.296 0)
+      (effects (font (size 1.27 1.27)) (justify right) hide)
+    )
+    (property "Footprint" "restall-generic-test:testpoint-SP3050A-with-short-gnd" (at 394.97 86.36 0)
+      (effects (font (size 1.27 1.27)) (justify right) hide)
+    )
+    (property "Datasheet" "~" (at 394.97 86.36 0)
+      (effects (font (size 1.27 1.27)) (justify right) hide)
+    )
+    (pin "2")
+    (pin "1")
+    (instances
+      (project "msf-owl-clock"
+        (path "/56d623d3-22db-4d43-a9d9-e6bb4bb68946/ce863d79-d266-4984-b56b-ca957df41c84/4fbb3fbf-2c3d-43d2-97c2-d56faba30b72"
+          (reference "TP209") (unit 1)
+        )
+      )
