File: src/schematics/2-msf-receiver-trf.kicad_sch (KiCad schematic)
At the start: 39 parts, among them U203 MCP6499, U204 MCP6499, U206 TMUX1511RSV, U207 TMUX1511RSV

Commit message: Added part numbers for the capacitors.
Parts:
- C233, C234, C239, C243, C244: ManufacturerPartNumber (none) -> CL05A475MP5NRNC
Changed lines of the file:
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@@
       (effects (font (size 1.27 1.27)) (justify left) hide)
     )
-    (property "ManufacturerPartNumber" "" (at 261.62 114.3 0)
+    (property "ManufacturerPartNumber" "CL05A475MP5NRNC" (at 261.62 114.3 0)
       (effects (font (size 1.27 1.27)) (justify left) hide)
     )
@@
       (effects (font (size 1.27 1.27)) (justify left) hide)
     )
-    (property "ManufacturerPartNumber" "" (at 38.1 149.86 0)
+    (property "ManufacturerPartNumber" "CL05A475MP5NRNC" (at 38.1 149.86 0)
       (effects (font (size 1.27 1.27)) (justify left) hide)
     )
@@
       (effects (font (size 1.27 1.27)) (justify left) hide)
     )
-    (property "ManufacturerPartNumber" "" (at 243.84 149.86 0)
+    (property "ManufacturerPartNumber" "CL05A475MP5NRNC" (at 243.84 149.86 0)
       (effects (font (size 1.27 1.27)) (justify left) hide)
     )
@@
       (effects (font (size 1.27 1.27)) (justify left) hide)
     )
-    (property "ManufacturerPartNumber" "" (at 63.5 114.3 0)
+    (property "ManufacturerPartNumber" "CL05A475MP5NRNC" (at 63.5 114.3 0)
       (effects (font (size 1.27 1.27)) (justify left) hide)
     )
@@
       (effects (font (size 1.27 1.27)) (justify left) hide)
     )
-    (property "ManufacturerPartNumber" "" (at 35.56 83.82 0)
-      (effects (font (size 1.27 1.27)) (justify left) hide)
-    )
+    (property "ManufacturerPartNumber" "CL05A475MP5NRNC" (at 35.56 83.82 0)
+      (effects (font (size 1.27 1.27)) (justify left) hide)
+    )
