File: src/schematics/2-msf-receiver-trf.kicad_sch (KiCad schematic)
At the start: 39 parts, among them U203 MCP6499, U204 MCP6499, U206 TMUX1511RSV, U207 TMUX1511RSV

Commit message: Added part numbers for the resistors.
Parts:
- R225, R227, R237: Manufacturer (none) -> Yageo; Manufacturer2 (none) -> Panasonic; Manufacturer2PartNumber (none) -> ERA-2AEB391X; ManufacturerPartNumber (none) -> RT0402BRD07390RL
- R226: Manufacturer (none) -> Panasonic; Manufacturer2 (none) -> Susumu; Manufacturer2PartNumber (none) -> RG1005P-470-B-T5; ManufacturerPartNumber (none) -> ERA-2AEB470X
- R228, R238: Manufacturer (none) -> Yageo; Manufacturer2 (none) -> Panasonic; Manufacturer2PartNumber (none) -> ERA-2AEB1241X; ManufacturerPartNumber (none) -> RT0402BRD071K24L
- R229, R235, R239: Manufacturer (none) -> Yageo; Manufacturer2 (none) -> Panasonic; Manufacturer2PartNumber (none) -> ERA-2AEB2491X; ManufacturerPartNumber (none) -> RT0402BRD072K49L
- R230, R240: Manufacturer (none) -> Yageo; Manufacturer2 (none) -> Vishay; Manufacturer2PartNumber (none) -> MCS04020D4991BE000; ManufacturerPartNumber (none) -> RT0402BRD074K99L
- R231, R241: Manufacturer (none) -> Yageo; Manufacturer2 (none) -> Panasonic; Manufacturer2PartNumber (none) -> ERA-2AEB4121X; ManufacturerPartNumber (none) -> RT0402BRD074K12L
- R232, R242: Manufacturer (none) -> TE Connectivity; Manufacturer2 (none) -> TE Connectivity; Manufacturer2PartNumber (none) -> CPF0402B64R9E1; ManufacturerPartNumber (none) -> RP73PF1E64R9BTD
- R233, R243: Manufacturer (none) -> Yageo; Manufacturer2 (none) -> Panasonic; Manufacturer2PartNumber (none) -> ERA-2AEB4992X; ManufacturerPartNumber (none) -> RT0402BRD0749K9L
- R234, R244: Manufacturer (none) -> Yageo; Manufacturer2 (none) -> Walsin; Manufacturer2PartNumber (none) -> WR04X000PTL; ManufacturerPartNumber (none) -> RC0402FR-070RL
- R236: Manufacturer (none) -> Yageo; Manufacturer2 (none) -> Yageo; Manufacturer2PartNumber (none) -> RT0402BRE07100RL; ManufacturerPartNumber (none) -> RT0402BRD07100RL

Commit message: Clean up the remaining ERC flags.
Parts:
- added NT201: Net Tie, restall-generic-wires:net-tie-2-6mil, symbol restall-generic-wires:net-tie-2
Connections:
- net MSF_ANT_{-}: now also NT201.1 (P1_PASSIVE); no longer C234.1, C239.1, R226.2, R235.2, R236.2, U203.12 (+), U204.10 (+)
- net FB0 renamed PGA1.FB0
- net PGA1.FB0: no longer C240.1, R236.1, R237.1, U204.6 (-), U207.10
- net FB1 renamed PGA1.FB1
- net PGA1.FB1: no longer R237.2, R238.1, U207.6, U207.9
- net FB2 renamed PGA1.FB2
- net PGA1.FB2: no longer R238.2, R239.1, U207.3, U207.5
- net FB3 renamed PGA1.FB3
- net PGA1.FB3: no longer R239.2, R240.1, U207.14, U207.2
- net FB4 renamed PGA1.FB4
- net PGA1.FB4: no longer C240.2, R240.2, R241.1, U204.7, U207.13
- net GND renamed GND_PWRIN
- net SW_EN0 renamed PGA1.SW_EN0
- net PGA1.SW_EN0: no longer U207.11
- net SW_EN1 renamed PGA1.SW_EN1
- net PGA1.SW_EN1: no longer U207.4
- net SW_EN2 renamed PGA1.SW_EN2
- net PGA1.SW_EN2: no longer U207.1
- net SW_EN3 renamed PGA1.SW_EN3
- net PGA1.SW_EN3: no longer U207.15
- new net MSF_RCV_VREF_{+1.8V}: C234.1, C239.1, NT201.2 (P2_PASSIVE), R226.2, R235.2, R236.2, U203.12 (+), U204.10 (+)
- new net PGA2.FB0: C240.1, R236.1, R237.1, U204.6 (-), U207.10
- new net PGA2.FB1: R237.2, R238.1, U207.6, U207.9
- new net PGA2.FB2: R238.2, R239.1, U207.3, U207.5
- new net PGA2.FB3: R239.2, R240.1, U207.14, U207.2
- new net PGA2.FB4: C240.2, R240.2, R241.1, U204.7, U207.13
- new net PGA2.SW_EN0: U207.11
- new net PGA2.SW_EN1: U207.4
- new net PGA2.SW_EN2: U207.1
- new net PGA2.SW_EN3: U207.15
Other:
- moved on the sheet: C243, U206A, U206B, U206C, U206D, U206E

Commit message: Started to lay out the PCB.
Connections:
- net GND_PWRIN renamed GND

Commit message: PCB routing.
Connections:
- net GND: no longer U206.7 (V_{SS}), U207.7 (V_{SS})

Commit message: PCB routing.
Connections:
- net MSF_RCV_TRF: now also U204.7; no longer U204.8
- net MSF_RCV_VREF_{+1.8V}: now also U204.5 (+); no longer U204.10 (+)
- net PGA2.FB0: now also U204.9 (-); no longer U204.6 (-)
- net PGA2.FB4: now also U204.8; no longer U204.7
- net at C242.2, R244.2: now also U204.6 (-); no longer U204.9 (-)
- net at C238.1, R235.1, TP208.1: now also U204.10 (+); no longer U204.5 (+)
Changed lines of the file:
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@@
     )
   )
-  (symbol (lib_id "restall-manufacturer-microchip:MCP6499?-?-S?") (at 374.65 78.74 0) (mirror x) (unit 3)
+  (symbol (lib_id "restall-manufacturer-microchip:MCP6499?-?-S?") (at 374.65 78.74 0) (mirror x) (unit 2)
     (in_bom yes) (on_board yes) (dnp no)
     (property "Reference" "U204" (at 368.554 77.724 0)
@@
       (project "msf-owl-clock"
         (path "/56d623d3-22db-4d43-a9d9-e6bb4bb68946/ce863d79-d266-4984-b56b-ca957df41c84/4fbb3fbf-2c3d-43d2-97c2-d56faba30b72"
-          (reference "U204") (unit 3)
+          (reference "U204") (unit 2)
         )
       )
@@
     )
   )
-  (symbol (lib_id "restall-manufacturer-microchip:MCP6499?-?-S?") (at 280.67 73.66 0) (unit 2)
+  (symbol (lib_id "restall-manufacturer-microchip:MCP6499?-?-S?") (at 280.67 73.66 0) (unit 3)
     (in_bom yes) (on_board yes) (dnp no)
     (property "Reference" "U204" (at 274.574 72.5861 0)
@@
       (project "msf-owl-clock"
         (path "/56d623d3-22db-4d43-a9d9-e6bb4bb68946/ce863d79-d266-4984-b56b-ca957df41c84/4fbb3fbf-2c3d-43d2-97c2-d56faba30b72"
-          (reference "U204") (unit 2)
+          (reference "U204") (unit 3)
         )
       )

Commit message: PCB routing.
Parts:
- removed NT201: Net Tie, restall-generic-wires:net-tie-2-6mil, symbol restall-generic-wires:net-tie-2
Connections:
- net MSF_RCV_VREF_{+1.8V} is gone; now on net MSF_ANT_{-}: C234.1, C239.1, R226.2, R235.2, R236.2, U203.12 (+), U204.5 (+)
Changed lines of the file:
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@@
   (junction (at 116.84 73.66) (diameter 0) (color 0 0 0 0)
   )
+  (junction (at 335.28 73.66) (diameter 0) (color 0 0 0 0)
+  )
+  (junction (at 294.64 152.4) (diameter 0) (color 0 0 0 0)
+  )
+  (junction (at 335.28 152.4) (diameter 0) (color 0 0 0 0)
+  )
+  (junction (at 187.96 78.74) (diameter 0) (color 0 0 0 0)
+  )
+  (junction (at 283.21 99.06) (diameter 0) (color 0 0 0 0)
+  )
+  (junction (at 71.12 68.58) (diameter 0) (color 0 0 0 0)
+  )
+  (junction (at 243.84 144.78) (diameter 0) (color 0 0 0 0)
+  )
+  (junction (at 63.5 86.36) (diameter 0) (color 0 0 0 0)
+  )
   (junction (at 35.56 78.74) (diameter 0) (color 0 0 0 0)
   )
-  (junction (at 335.28 73.66) (diameter 0) (color 0 0 0 0)
-  )
-  (junction (at 294.64 152.4) (diameter 0) (color 0 0 0 0)
-  )
-  (junction (at 335.28 152.4) (diameter 0) (color 0 0 0 0)
-  )
-  (junction (at 187.96 78.74) (diameter 0) (color 0 0 0 0)
-  )
-  (junction (at 283.21 99.06) (diameter 0) (color 0 0 0 0)
-  )
-  (junction (at 71.12 68.58) (diameter 0) (color 0 0 0 0)
-  )
-  (junction (at 243.84 144.78) (diameter 0) (color 0 0 0 0)
-  )
-  (junction (at 63.5 86.36) (diameter 0) (color 0 0 0 0)
-  )
   (junction (at 137.16 73.66) (diameter 0) (color 0 0 0 0)
   )
@@
     (stroke (width 0) (type default))
   )
-  (wire (pts (xy 38.1 78.74) (xy 48.26 78.74))
+  (wire (pts (xy 33.02 78.74) (xy 35.56 78.74))
     (stroke (width 0) (type default))
   )
@@
     (stroke (width 0) (type default))
   )
+  (wire (pts (xy 35.56 78.74) (xy 48.26 78.74))
+    (stroke (width 0) (type default))
+  )
   (wire (pts (xy 154.94 50.8) (xy 187.96 50.8))
     (stroke (width 0) (type default))
@@
   )
   (wire (pts (xy 363.22 83.82) (xy 365.76 83.82))
-    (stroke (width 0) (type default))
-  )
-  (wire (pts (xy 33.02 78.74) (xy 35.56 78.74))
     (stroke (width 0) (type default))
   )
@@
         )
       )
-    )
-  )
-  (symbol (lib_id "restall-generic-wires:net-tie-2") (at 36.83 78.74 0) (unit 1)
-    (in_bom no) (on_board yes) (dnp no) (fields_autoplaced)
-    (property "Reference" "NT201" (at 36.83 76.2 0)
-      (effects (font (size 1.27 1.27)) hide)
-    )
-    (property "Value" "Net Tie" (at 36.83 81.28 0)
-      (effects (font (size 1.27 1.27)) hide)
-    )
-    (property "Footprint" "restall-generic-wires:net-tie-2-6mil" (at 36.83 83.312 0)
-      (effects (font (size 1.27 1.27)) hide)
-    )
-    (property "Datasheet" "~" (at 36.83 85.344 0)
-      (effects (font (size 1.27 1.27)) hide)
-    )
-    (pin "1")
-    (pin "2")
-    (instances
-      (project "msf-owl-clock"
-        (path "/56d623d3-22db-4d43-a9d9-e6bb4bb68946/ce863d79-d266-4984-b56b-ca957df41c84/4fbb3fbf-2c3d-43d2-97c2-d56faba30b72"
-          (reference "NT201") (unit 1)
-        )
-      )

Commit message: PCB routing.
Parts:
- added TP210: ~, restall-generic-test:testpoint-SP3050A-with-short-gnd, symbol restall-generic-test:testpoint-probe-with-gnd
Connections:
- net GND: now also TP210.2 (GND)
- net MSF_ANT_{-}: now also TP210.1
Changed lines of the file:
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@@
   (junction (at 48.26 109.22) (diameter 0) (color 0 0 0 0)
   )
+  (junction (at 41.91 109.22) (diameter 0) (color 0 0 0 0)
+  )
   (bus_entry (at 316.23 106.68) (size -2.54 -2.54)
     (stroke (width 0) (type default))
@@
     (stroke (width 0) (type default))
   )
-  (wire (pts (xy 33.02 109.22) (xy 48.26 109.22))
-    (stroke (width 0) (type default))
-  )
   (bus (pts (xy 127 162.56) (xy 147.32 162.56))
     (stroke (width 0) (type default))
@@
     (stroke (width 0) (type default))
   )
+  (wire (pts (xy 33.02 109.22) (xy 41.91 109.22))
+    (stroke (width 0) (type default))
+  )
   (wire (pts (xy 129.54 85.09) (xy 129.54 83.82))
     (stroke (width 0) (type default))
@@
     (stroke (width 0) (type default))
   )
+  (wire (pts (xy 41.91 102.87) (xy 41.91 109.22))
+    (stroke (width 0) (type default))
+  )
   (wire (pts (xy 186.69 78.74) (xy 187.96 78.74))
     (stroke (width 0) (type default))
@@
   )
   (bus (pts (xy 238.76 162.56) (xy 284.48 162.56))
+    (stroke (width 0) (type default))
+  )
+  (wire (pts (xy 41.91 109.22) (xy 48.26 109.22))
     (stroke (width 0) (type default))
   )
@@
     )
   )
+  (symbol (lib_id "restall-generic-test:testpoint-probe-with-gnd") (at 41.91 102.87 0) (mirror y) (unit 1)
+    (in_bom no) (on_board yes) (dnp no)
+    (property "Reference" "TP210" (at 32.258 100.33 0)
+      (effects (font (size 1.27 1.27)) (justify right))
+    )
+    (property "Value" "~" (at 40.259 98.806 0)
+      (effects (font (size 1.27 1.27)) (justify right) hide)
+    )
+    (property "Footprint" "restall-generic-test:testpoint-SP3050A-with-short-gnd" (at 36.83 102.87 0)
+      (effects (font (size 1.27 1.27)) (justify right) hide)
+    )
+    (property "Datasheet" "~" (at 36.83 102.87 0)
+      (effects (font (size 1.27 1.27)) (justify right) hide)
+    )
+    (pin "2")
+    (pin "1")
+    (instances
+      (project "msf-owl-clock"
+        (path "/56d623d3-22db-4d43-a9d9-e6bb4bb68946/ce863d79-d266-4984-b56b-ca957df41c84/4fbb3fbf-2c3d-43d2-97c2-d56faba30b72"
+          (reference "TP210") (unit 1)
+        )
+      )
+    )
+  )
   (symbol (lib_id "restall-generic-power:GND") (at 63.5 118.11 0) (unit 1)
     (in_bom yes) (on_board yes) (dnp no) (fields_autoplaced)
@@
         )
       )
+    )
+  )
+  (symbol (lib_id "restall-generic-power:GND") (at 38.862 102.87 0) (unit 1)
+    (in_bom yes) (on_board yes) (dnp no) (fields_autoplaced)
+    (property "Reference" "#PWR0281" (at 38.862 109.22 0)
+      (effects (font (size 1.27 1.27)) hide)
+    )
+    (property "Value" "GND" (at 38.862 107.0031 0)
+      (effects (font (size 1.27 1.27)))
+    )
+    (property "Footprint" "" (at 38.862 102.87 0)
+      (effects (font (size 1.27 1.27)) hide)
+    )
+    (property "Datasheet" "" (at 38.862 102.87 0)
+      (effects (font (size 1.27 1.27)) hide)
+    )
+    (pin "1")
+    (instances
+      (project "msf-owl-clock"
+        (path "/56d623d3-22db-4d43-a9d9-e6bb4bb68946/ce863d79-d266-4984-b56b-ca957df41c84/4fbb3fbf-2c3d-43d2-97c2-d56faba30b72"
+          (reference "#PWR0281") (unit 1)
+        )
+      )

Commit message: PCB routing.  Fixed most of the DRC violations.
Connections:
- net GND: no longer U206.12 (NC), U207.12 (NC)
Changed lines of the file:
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@@
     (pin "8")
     (pin "9")
-    (pin "12")
+    (pin "12" (alternate "NC-NC"))
     (pin "13")
     (pin "16")
@@
     (pin "8")
     (pin "9")
-    (pin "12")
+    (pin "12" (alternate "NC-NC"))
     (pin "13")
     (pin "16")
@@
     (pin "8")
     (pin "9")
-    (pin "12")
+    (pin "12" (alternate "NC-NC"))
     (pin "13")
     (pin "16")
@@
     (pin "8")
     (pin "9")
-    (pin "12")
+    (pin "12" (alternate "NC-NC"))
     (pin "13")
     (pin "16")
@@
     (pin "8")
     (pin "9")
-    (pin "12")
+    (pin "12" (alternate "NC-NC"))
     (pin "13")
     (pin "16")
@@
     (pin "8")
     (pin "9")
-    (pin "12")
+    (pin "12" (alternate "NC-NC"))
     (pin "13")
     (pin "16")
@@
     (pin "8")
     (pin "9")
-    (pin "12")
+    (pin "12" (alternate "NC-NC"))
     (pin "13")
     (pin "16")
@@
     (pin "8")
     (pin "9")
-    (pin "12")
+    (pin "12" (alternate "NC-NC"))
     (pin "13")
     (pin "16")
@@
     (pin "8")
     (pin "9")
-    (pin "12")
+    (pin "12" (alternate "NC-NC"))
     (pin "13")
     (pin "16")
@@
     (pin "8")
     (pin "9")
-    (pin "12")
+    (pin "12" (alternate "NC-NC"))
     (pin "13")
     (pin "16")
