File: src/schematics/2-msf-receiver-trf.kicad_sch (KiCad schematic)
At the start: 40 parts, among them U203 MCP6499, U204 MCP6499, U206 TMUX1511RSV, U207 TMUX1511RSV

Commit message: Final push to JLCPCB.  Fixed various component rotation mismatches, some silkscreen issues, BOM amendments due to component availability, etc.
Parts:
- C236, C238, C241: Manufacturer Yageo -> Murata; Manufacturer2 Murata -> Yageo; Manufacturer2PartNumber GCM1885C1H472GA16D -> CC0603FRNPO9BN472; ManufacturerPartNumber CC0603FRNPO9BN472 -> GCM1885C1H472GA16D
Changed lines of the file:
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@@
       (effects (font (size 1.27 1.27)) (justify left))
     )
-    (property "Manufacturer" "Yageo" (at 245.11 68.58 0)
-      (effects (font (size 1.27 1.27)) (justify right) hide)
-    )
-    (property "ManufacturerPartNumber" "CC0603FRNPO9BN472" (at 245.11 68.58 0)
-      (effects (font (size 1.27 1.27)) (justify right) hide)
-    )
-    (property "Manufacturer2" "Murata" (at 245.11 68.58 0)
-      (effects (font (size 1.27 1.27)) (justify right) hide)
-    )
-    (property "Manufacturer2PartNumber" "GCM1885C1H472GA16D" (at 245.11 68.58 0)
+    (property "Manufacturer" "Murata" (at 245.11 68.58 0)
+      (effects (font (size 1.27 1.27)) (justify right) hide)
+    )
+    (property "ManufacturerPartNumber" "GCM1885C1H472GA16D" (at 245.11 68.58 0)
+      (effects (font (size 1.27 1.27)) (justify right) hide)
+    )
+    (property "Manufacturer2" "Yageo" (at 245.11 68.58 0)
+      (effects (font (size 1.27 1.27)) (justify right) hide)
+    )
+    (property "Manufacturer2PartNumber" "CC0603FRNPO9BN472" (at 245.11 68.58 0)
       (effects (font (size 1.27 1.27)) (justify right) hide)
     )
@@
       (effects (font (size 1.27 1.27)) (justify right))
     )
-    (property "Manufacturer" "Yageo" (at 137.16 57.15 0)
-      (effects (font (size 1.27 1.27)) (justify right) hide)
-    )
-    (property "ManufacturerPartNumber" "CC0603FRNPO9BN472" (at 137.16 57.15 0)
-      (effects (font (size 1.27 1.27)) (justify right) hide)
-    )
-    (property "Manufacturer2" "Murata" (at 137.16 57.15 0)
-      (effects (font (size 1.27 1.27)) (justify right) hide)
-    )
-    (property "Manufacturer2PartNumber" "GCM1885C1H472GA16D" (at 137.16 57.15 0)
+    (property "Manufacturer" "Murata" (at 137.16 57.15 0)
+      (effects (font (size 1.27 1.27)) (justify right) hide)
+    )
+    (property "ManufacturerPartNumber" "GCM1885C1H472GA16D" (at 137.16 57.15 0)
+      (effects (font (size 1.27 1.27)) (justify right) hide)
+    )
+    (property "Manufacturer2" "Yageo" (at 137.16 57.15 0)
+      (effects (font (size 1.27 1.27)) (justify right) hide)
+    )
+    (property "Manufacturer2PartNumber" "CC0603FRNPO9BN472" (at 137.16 57.15 0)
       (effects (font (size 1.27 1.27)) (justify right) hide)
     )
@@
       (effects (font (size 1.27 1.27)) (justify right))
     )
-    (property "Manufacturer" "Yageo" (at 335.28 57.15 0)
-      (effects (font (size 1.27 1.27)) (justify right) hide)
-    )
-    (property "ManufacturerPartNumber" "CC0603FRNPO9BN472" (at 335.28 57.15 0)
-      (effects (font (size 1.27 1.27)) (justify right) hide)
-    )
-    (property "Manufacturer2" "Murata" (at 335.28 57.15 0)
-      (effects (font (size 1.27 1.27)) (justify right) hide)
-    )
-    (property "Manufacturer2PartNumber" "GCM1885C1H472GA16D" (at 335.28 57.15 0)
-      (effects (font (size 1.27 1.27)) (justify right) hide)
-    )
+    (property "Manufacturer" "Murata" (at 335.28 57.15 0)
+      (effects (font (size 1.27 1.27)) (justify right) hide)
+    )
+    (property "ManufacturerPartNumber" "GCM1885C1H472GA16D" (at 335.28 57.15 0)
+      (effects (font (size 1.27 1.27)) (justify right) hide)
+    )
+    (property "Manufacturer2" "Yageo" (at 335.28 57.15 0)
+      (effects (font (size 1.27 1.27)) (justify right) hide)
+    )
+    (property "Manufacturer2PartNumber" "CC0603FRNPO9BN472" (at 335.28 57.15 0)
+      (effects (font (size 1.27 1.27)) (justify right) hide)
+    )
