File: src/schematics/msf-owl-clock.kicad_sch (KiCad schematic)
At the start: 56 parts, among them U001 BC805M, U002 TSOP75338TT

Commit message: Added part numbers for the capacitors.
Parts:
- C001, C004, C005, C006, C007, C008, C009, C010: ManufacturerPartNumber (none) -> CL05A475MP5NRNC
- C011: Manufacturer (none) -> Samsung; Manufacturer2 (none) -> Samsung; Manufacturer2PartNumber (none) -> CL05A104KA5NNNC; ManufacturerPartNumber (none) -> CL05B104KA5NNNC
- CONN001: Package (none) -> GSB1CA11101DSHR
- FB001: Package (none) -> WLBD2012
- SPK001: Package (none) -> 502443-0270
Changed lines of the file:
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@@
       (effects (font (size 1.27 1.27)) (justify left) hide)
     )
-    (property "ManufacturerPartNumber" "" (at 325.12 25.4 0)
+    (property "ManufacturerPartNumber" "CL05A475MP5NRNC" (at 325.12 25.4 0)
       (effects (font (size 1.27 1.27)) (justify left) hide)
     )
@@
       (effects (font (size 1.27 1.27)) (justify left) hide)
     )
-    (property "Manufacturer" "" (at 17.78 76.2 0)
+    (property "Manufacturer" "Samsung" (at 17.78 76.2 0)
       (effects (font (size 1.27 1.27)) (justify left) hide)
     )
-    (property "ManufacturerPartNumber" "" (at 17.78 76.2 0)
+    (property "ManufacturerPartNumber" "CL05B104KA5NNNC" (at 17.78 76.2 0)
       (effects (font (size 1.27 1.27)) (justify left) hide)
     )
-    (property "Manufacturer2" "" (at 17.78 76.2 0)
+    (property "Manufacturer2" "Samsung" (at 17.78 76.2 0)
       (effects (font (size 1.27 1.27)) (justify left) hide)
     )
-    (property "Manufacturer2PartNumber" "" (at 17.78 76.2 0)
+    (property "Manufacturer2PartNumber" "CL05A104KA5NNNC" (at 17.78 76.2 0)
       (effects (font (size 1.27 1.27)) (justify left) hide)
     )
@@
       (effects (font (size 1.27 1.27)) (justify left) hide)
     )
-    (property "ManufacturerPartNumber" "" (at 312.42 25.4 0)
+    (property "ManufacturerPartNumber" "CL05A475MP5NRNC" (at 312.42 25.4 0)
       (effects (font (size 1.27 1.27)) (justify left) hide)
     )
@@
       (effects (font (size 1.27 1.27)) (justify left) hide)
     )
+    (property "Package" "502443-0270" (at 373.38 194.31 0)
+      (effects (font (size 1.27 1.27)) hide)
+    )
     (pin "2")
     (pin "1")
@@
       (effects (font (size 1.27 1.27)) (justify left) hide)
     )
-    (property "ManufacturerPartNumber" "" (at 233.68 25.4 0)
+    (property "ManufacturerPartNumber" "CL05A475MP5NRNC" (at 233.68 25.4 0)
       (effects (font (size 1.27 1.27)) (justify left) hide)
     )
@@
       (effects (font (size 1.27 1.27)) (justify left) hide)
     )
-    (property "ManufacturerPartNumber" "" (at 220.98 25.4 0)
+    (property "ManufacturerPartNumber" "CL05A475MP5NRNC" (at 220.98 25.4 0)
       (effects (font (size 1.27 1.27)) (justify left) hide)
     )
@@
       (effects (font (size 1.27 1.27)) (justify left) hide)
     )
-    (property "ManufacturerPartNumber" "" (at 363.22 55.88 0)
+    (property "ManufacturerPartNumber" "CL05A475MP5NRNC" (at 363.22 55.88 0)
       (effects (font (size 1.27 1.27)) (justify left) hide)
     )
@@
       (effects (font (size 1.27 1.27)) (justify left))
     )
+    (property "Package" "GSB1CA11101DSHR" (at 38.1 102.87 0)
+      (effects (font (size 1.27 1.27)) hide)
+    )
     (pin "B7")
     (pin "B4")
@@
       (effects (font (size 1.27 1.27)) (justify left) hide)
     )
+    (property "Package" "WLBD2012" (at 137.16 20.32 0)
+      (effects (font (size 1.27 1.27)) hide)
+    )
     (pin "1")
     (pin "2")
@@
       (effects (font (size 1.27 1.27)) (justify left) hide)
     )
-    (property "ManufacturerPartNumber" "" (at 101.6 25.4 0)
+    (property "ManufacturerPartNumber" "CL05A475MP5NRNC" (at 101.6 25.4 0)
       (effects (font (size 1.27 1.27)) (justify left) hide)
     )
@@
       (effects (font (size 1.27 1.27)) (justify left) hide)
     )
-    (property "ManufacturerPartNumber" "" (at 246.38 25.4 0)
+    (property "ManufacturerPartNumber" "CL05A475MP5NRNC" (at 246.38 25.4 0)
       (effects (font (size 1.27 1.27)) (justify left) hide)
     )
@@
       (effects (font (size 1.27 1.27)) (justify left) hide)
     )
-    (property "ManufacturerPartNumber" "" (at 299.72 25.4 0)
+    (property "ManufacturerPartNumber" "CL05A475MP5NRNC" (at 299.72 25.4 0)
       (effects (font (size 1.27 1.27)) (justify left) hide)
     )
