File: src/schematics/4-audio-out.kicad_sch (KiCad schematic)
At the start: 34 parts, among them U401 AP22653AW6, U402 MCP6486U, U403 IS31AP4991A-SLS2

Commit message: Added part numbers for the resistors.
Parts:
- R401, R402: Manufacturer (none) -> Walsin; Manufacturer2 (none) -> Yageo; Manufacturer2PartNumber (none) -> RC0402FR-0733KL; ManufacturerPartNumber (none) -> WR04X3302FTL
- R403: Manufacturer (none) -> KOA Speer; Manufacturer2 (none) -> Yageo; Manufacturer2PartNumber (none) -> RT0402BRD0768KL; ManufacturerPartNumber (none) -> RN73R1ETTP6802B25
- R404, R408, R409: Manufacturer (none) -> Walsin; Manufacturer2 (none) -> Yageo; Manufacturer2PartNumber (none) -> RC0402FR-0719K6L; ManufacturerPartNumber (none) -> WR04X1962FTL
- R405: Manufacturer (none) -> Walsin; Manufacturer2 (none) -> Yageo; Manufacturer2PartNumber (none) -> RC0402FR-075K1L; ManufacturerPartNumber (none) -> WR04X5101FTL
- R406: Manufacturer (none) -> Yageo; Manufacturer2 (none) -> Panasonic; Manufacturer2PartNumber (none) -> ERJ2RKF1602X; ManufacturerPartNumber (none) -> AC0402DR-0716KL
- R407: Manufacturer (none) -> Yageo; Manufacturer2 (none) -> Yageo; Manufacturer2PartNumber (none) -> AC0402DR-0739KL; ManufacturerPartNumber (none) -> RC0402FR-0739KL
Changed lines of the file:
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@@
       (effects (font (size 1.27 1.27)) (justify left) hide)
     )
-    (property "Manufacturer" "" (at 149.86 88.9 0)
-      (effects (font (size 1.27 1.27)) (justify left) hide)
-    )
-    (property "ManufacturerPartNumber" "" (at 149.86 88.9 0)
-      (effects (font (size 1.27 1.27)) (justify left) hide)
-    )
-    (property "Manufacturer2" "" (at 149.86 88.9 0)
-      (effects (font (size 1.27 1.27)) (justify left) hide)
-    )
-    (property "Manufacturer2PartNumber" "" (at 149.86 88.9 0)
+    (property "Manufacturer" "KOA Speer" (at 149.86 88.9 0)
+      (effects (font (size 1.27 1.27)) (justify left) hide)
+    )
+    (property "ManufacturerPartNumber" "RN73R1ETTP6802B25" (at 149.86 88.9 0)
+      (effects (font (size 1.27 1.27)) (justify left) hide)
+    )
+    (property "Manufacturer2" "Yageo" (at 149.86 88.9 0)
+      (effects (font (size 1.27 1.27)) (justify left) hide)
+    )
+    (property "Manufacturer2PartNumber" "RT0402BRD0768KL" (at 149.86 88.9 0)
       (effects (font (size 1.27 1.27)) (justify left) hide)
     )
@@
       (effects (font (size 1.27 1.27)) (justify left) hide)
     )
-    (property "Manufacturer" "" (at 151.13 147.32 0)
-      (effects (font (size 1.27 1.27)) (justify left) hide)
-    )
-    (property "ManufacturerPartNumber" "" (at 151.13 147.32 0)
-      (effects (font (size 1.27 1.27)) (justify left) hide)
-    )
-    (property "Manufacturer2" "" (at 151.13 147.32 0)
-      (effects (font (size 1.27 1.27)) (justify left) hide)
-    )
-    (property "Manufacturer2PartNumber" "" (at 151.13 147.32 0)
+    (property "Manufacturer" "Walsin" (at 151.13 147.32 0)
+      (effects (font (size 1.27 1.27)) (justify left) hide)
+    )
+    (property "ManufacturerPartNumber" "WR04X1962FTL" (at 151.13 147.32 0)
+      (effects (font (size 1.27 1.27)) (justify left) hide)
+    )
+    (property "Manufacturer2" "Yageo" (at 151.13 147.32 0)
+      (effects (font (size 1.27 1.27)) (justify left) hide)
+    )
+    (property "Manufacturer2PartNumber" "RC0402FR-0719K6L" (at 151.13 147.32 0)
       (effects (font (size 1.27 1.27)) (justify left) hide)
     )
@@
       (effects (font (size 1.27 1.27)) (justify left) hide)
     )
-    (property "Manufacturer" "" (at 137.16 89.154 0)
-      (effects (font (size 1.27 1.27)) (justify left) hide)
-    )
-    (property "ManufacturerPartNumber" "" (at 137.16 89.154 0)
-      (effects (font (size 1.27 1.27)) (justify left) hide)
-    )
-    (property "Manufacturer2" "" (at 137.16 89.154 0)
-      (effects (font (size 1.27 1.27)) (justify left) hide)
-    )
-    (property "Manufacturer2PartNumber" "" (at 137.16 89.154 0)
+    (property "Manufacturer" "Walsin" (at 137.16 89.154 0)
+      (effects (font (size 1.27 1.27)) (justify left) hide)
+    )
+    (property "ManufacturerPartNumber" "WR04X3302FTL" (at 137.16 89.154 0)
+      (effects (font (size 1.27 1.27)) (justify left) hide)
+    )
+    (property "Manufacturer2" "Yageo" (at 137.16 89.154 0)
+      (effects (font (size 1.27 1.27)) (justify left) hide)
+    )
+    (property "Manufacturer2PartNumber" "RC0402FR-0733KL" (at 137.16 89.154 0)
       (effects (font (size 1.27 1.27)) (justify left) hide)
     )
@@
       (effects (font (size 1.27 1.27)) (justify left) hide)
     )
-    (property "Manufacturer" "" (at 182.88 121.92 0)
-      (effects (font (size 1.27 1.27)) (justify left) hide)
-    )
-    (property "ManufacturerPartNumber" "" (at 182.88 121.92 0)
-      (effects (font (size 1.27 1.27)) (justify left) hide)
-    )
-    (property "Manufacturer2" "" (at 182.88 121.92 0)
-      (effects (font (size 1.27 1.27)) (justify left) hide)
-    )
-    (property "Manufacturer2PartNumber" "" (at 182.88 121.92 0)
+    (property "Manufacturer" "Yageo" (at 182.88 121.92 0)
+      (effects (font (size 1.27 1.27)) (justify left) hide)
+    )
+    (property "ManufacturerPartNumber" "RC0402FR-0739KL" (at 182.88 121.92 0)
+      (effects (font (size 1.27 1.27)) (justify left) hide)
+    )
+    (property "Manufacturer2" "Yageo" (at 182.88 121.92 0)
+      (effects (font (size 1.27 1.27)) (justify left) hide)
+    )
+    (property "Manufacturer2PartNumber" "AC0402DR-0739KL" (at 182.88 121.92 0)
       (effects (font (size 1.27 1.27)) (justify left) hide)
     )
@@
       (effects (font (size 1.27 1.27)) (justify left) hide)
     )
-    (property "Manufacturer" "" (at 229.87 152.4 0)
-      (effects (font (size 1.27 1.27)) (justify left) hide)
-    )
-    (property "ManufacturerPartNumber" "" (at 229.87 152.4 0)
-      (effects (font (size 1.27 1.27)) (justify left) hide)
-    )
-    (property "Manufacturer2" "" (at 229.87 152.4 0)
-      (effects (font (size 1.27 1.27)) (justify left) hide)
-    )
-    (property "Manufacturer2PartNumber" "" (at 229.87 152.4 0)
+    (property "Manufacturer" "Walsin" (at 229.87 152.4 0)
+      (effects (font (size 1.27 1.27)) (justify left) hide)
+    )
+    (property "ManufacturerPartNumber" "WR04X1962FTL" (at 229.87 152.4 0)
+      (effects (font (size 1.27 1.27)) (justify left) hide)
+    )
+    (property "Manufacturer2" "Yageo" (at 229.87 152.4 0)
+      (effects (font (size 1.27 1.27)) (justify left) hide)
+    )
+    (property "Manufacturer2PartNumber" "RC0402FR-0719K6L" (at 229.87 152.4 0)
       (effects (font (size 1.27 1.27)) (justify left) hide)
     )
@@
       (effects (font (size 1.27 1.27)) (justify left) hide)
     )
-    (property "Manufacturer" "" (at 124.46 88.9 0)
-      (effects (font (size 1.27 1.27)) (justify left) hide)
-    )
-    (property "ManufacturerPartNumber" "" (at 124.46 88.9 0)
-      (effects (font (size 1.27 1.27)) (justify left) hide)
-    )
-    (property "Manufacturer2" "" (at 124.46 88.9 0)
-      (effects (font (size 1.27 1.27)) (justify left) hide)
-    )
-    (property "Manufacturer2PartNumber" "" (at 124.46 88.9 0)
+    (property "Manufacturer" "Walsin" (at 124.46 88.9 0)
+      (effects (font (size 1.27 1.27)) (justify left) hide)
+    )
+    (property "ManufacturerPartNumber" "WR04X3302FTL" (at 124.46 88.9 0)
+      (effects (font (size 1.27 1.27)) (justify left) hide)
+    )
+    (property "Manufacturer2" "Yageo" (at 124.46 88.9 0)
+      (effects (font (size 1.27 1.27)) (justify left) hide)
+    )
+    (property "Manufacturer2PartNumber" "RC0402FR-0733KL" (at 124.46 88.9 0)
       (effects (font (size 1.27 1.27)) (justify left) hide)
     )
@@
       (effects (font (size 1.27 1.27)) (justify left) hide)
     )
-    (property "Manufacturer" "" (at 171.45 147.32 0)
-      (effects (font (size 1.27 1.27)) (justify left) hide)
-    )
-    (property "ManufacturerPartNumber" "" (at 171.45 147.32 0)
-      (effects (font (size 1.27 1.27)) (justify left) hide)
-    )
-    (property "Manufacturer2" "" (at 171.45 147.32 0)
-      (effects (font (size 1.27 1.27)) (justify left) hide)
-    )
-    (property "Manufacturer2PartNumber" "" (at 171.45 147.32 0)
+    (property "Manufacturer" "Yageo" (at 171.45 147.32 0)
+      (effects (font (size 1.27 1.27)) (justify left) hide)
+    )
+    (property "ManufacturerPartNumber" "AC0402DR-0716KL" (at 171.45 147.32 0)
+      (effects (font (size 1.27 1.27)) (justify left) hide)
+    )
+    (property "Manufacturer2" "Panasonic" (at 171.45 147.32 0)
+      (effects (font (size 1.27 1.27)) (justify left) hide)
+    )
+    (property "Manufacturer2PartNumber" "ERJ2RKF1602X" (at 171.45 147.32 0)
       (effects (font (size 1.27 1.27)) (justify left) hide)
     )
@@
       (effects (font (size 1.27 1.27)) (justify left) hide)
     )
-    (property "Manufacturer" "" (at 161.29 147.32 0)
-      (effects (font (size 1.27 1.27)) (justify left) hide)
-    )
-    (property "ManufacturerPartNumber" "" (at 161.29 147.32 0)
-      (effects (font (size 1.27 1.27)) (justify left) hide)
-    )
-    (property "Manufacturer2" "" (at 161.29 147.32 0)
-      (effects (font (size 1.27 1.27)) (justify left) hide)
-    )
-    (property "Manufacturer2PartNumber" "" (at 161.29 147.32 0)
+    (property "Manufacturer" "Walsin" (at 161.29 147.32 0)
+      (effects (font (size 1.27 1.27)) (justify left) hide)
+    )
+    (property "ManufacturerPartNumber" "WR04X5101FTL" (at 161.29 147.32 0)
+      (effects (font (size 1.27 1.27)) (justify left) hide)
+    )
+    (property "Manufacturer2" "Yageo" (at 161.29 147.32 0)
+      (effects (font (size 1.27 1.27)) (justify left) hide)
+    )
+    (property "Manufacturer2PartNumber" "RC0402FR-075K1L" (at 161.29 147.32 0)
       (effects (font (size 1.27 1.27)) (justify left) hide)
     )
@@
       (effects (font (size 1.27 1.27)) (justify left) hide)
     )
-    (property "Manufacturer" "" (at 243.84 139.7 0)
-      (effects (font (size 1.27 1.27)) (justify left) hide)
-    )
-    (property "ManufacturerPartNumber" "" (at 243.84 139.7 0)
-      (effects (font (size 1.27 1.27)) (justify left) hide)
-    )
-    (property "Manufacturer2" "" (at 243.84 139.7 0)
-      (effects (font (size 1.27 1.27)) (justify left) hide)
-    )
-    (property "Manufacturer2PartNumber" "" (at 243.84 139.7 0)
-      (effects (font (size 1.27 1.27)) (justify left) hide)
-    )
+    (property "Manufacturer" "Walsin" (at 243.84 139.7 0)
+      (effects (font (size 1.27 1.27)) (justify left) hide)
+    )
+    (property "ManufacturerPartNumber" "WR04X1962FTL" (at 243.84 139.7 0)
+      (effects (font (size 1.27 1.27)) (justify left) hide)
+    )
+    (property "Manufacturer2" "Yageo" (at 243.84 139.7 0)
+      (effects (font (size 1.27 1.27)) (justify left) hide)
+    )
+    (property "Manufacturer2PartNumber" "RC0402FR-0719K6L" (at 243.84 139.7 0)
+      (effects (font (size 1.27 1.27)) (justify left) hide)
+    )

Commit message: Clean up the remaining ERC flags.
Connections:
- net GND renamed GND_PWRIN
Changed lines of the file:
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@@
       (effects (font (size 1.27 1.27)) hide)
     )
-    (pin "1")
-    (pin "2")
+    (pin "1" (alternate "P1_PWRIN"))
+    (pin "2" (alternate "P2_PWROUT"))
     (instances
       (project "msf-owl-clock"
