File: src/schematics/5-sensors.kicad_sch (KiCad schematic)
At the start: 36 parts, among them Q501 NX6008NBKW, Q502 NX6008NBKW, Q503 NX6008NBKW, Q504 NX6008NBKW, Q505 NX6008NBKW, U501 TPS7A2028PDBVR, U502 DPS310XTSA1, U503 HDC3022, U504 VL6180V1NR1

Commit message: Clean up the remaining ERC flags.
Connections:
- net GND renamed GND_PWRIN

Commit message: Started to lay out the PCB.
Connections:
- net GND_PWRIN renamed GND
