File: src/schematics/5-sensors.kicad_sch (KiCad schematic)
At the start: 36 parts, among them Q501 NX6008NBKW, Q502 NX6008NBKW, Q503 NX6008NBKW, Q504 NX6008NBKW, Q505 NX6008NBKW, U501 TPS7A2028PDBVR, U502 DPS310XTSA1, U503 HDC3022, U504 VL6180V1NR1

Commit message: Added part numbers for the resistors.
Parts:
- R501, R502, R507, R508, R509, R512, R513: Manufacturer (none) -> Walsin; Manufacturer2 (none) -> Yageo; Manufacturer2PartNumber (none) -> RC0402FR-0733KL; ManufacturerPartNumber (none) -> WR04X3302FTL
- R503, R504, R510, R511: Manufacturer (none) -> Walsin; Manufacturer2 (none) -> Yageo; Manufacturer2PartNumber (none) -> RC0402FR-07100RL; ManufacturerPartNumber (none) -> WR04X1000FTL
- R505, R506: Manufacturer (none) -> Yageo; Manufacturer2 (none) -> Walsin; Manufacturer2PartNumber (none) -> MR04X1801FTL; ManufacturerPartNumber (none) -> RC0402FR-071K8L

Commit message: Started to clean up the ERC flags.
Connections:
- now unconnected: U504.11 (NC), U504.2 (NC), U504.3 (NC), U504.7 (NC)

Commit message: PCB routing.
Parts:
- TP502, TP503: footprint restall-generic-test:testpoint-SP3050A-with-short-gnd -> restall-generic-test:th-testpoint-0.5mm-with-short-gnd
Changed lines of the file:
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@@
       (effects (font (size 1.27 1.27)) (justify right) hide)
     )
-    (property "Footprint" "restall-generic-test:testpoint-SP3050A-with-short-gnd" (at 165.608 259.08 0)
+    (property "Footprint" "restall-generic-test:th-testpoint-0.5mm-with-short-gnd" (at 165.608 259.08 0)
       (effects (font (size 1.27 1.27)) (justify right) hide)
     )
@@
       (effects (font (size 1.27 1.27)) (justify right) hide)
     )
-    (property "Footprint" "restall-generic-test:testpoint-SP3050A-with-short-gnd" (at 165.608 248.92 0)
+    (property "Footprint" "restall-generic-test:th-testpoint-0.5mm-with-short-gnd" (at 165.608 248.92 0)
       (effects (font (size 1.27 1.27)) (justify right) hide)
     )
