File: src/schematics/msf-owl-clock.kicad_pcb (KiCad board)
At the start: 4 copper layers, 130.1 x 183.6 mm, 446 parts, among them Q101 NX6008NBKW, Q301 NX6008NBKW, Q501 NX6008NBKW, Q502 NX6008NBKW, Q503 NX6008NBKW, Q504 NX6008NBKW, Q505 NX6008NBKW, Q601 NX6008NBKW, Q602 BC847BS, Q603 BC847BS, U001 BC805M, U002 TSOP75338TT, U101 MP5016HGQH, U102 BQ24392RSER, U103 FUSB302BMPX, U104 TPS628512DRLR, U201 TPS7A2040PDQNR, U202 TPS7A2036PDBVR, U203 MCP6499, U204 MCP6499, U205 74HC595BQ, U206 TMUX1511RSV, U207 TMUX1511RSV, U301 PIC32CX1025SG41100-I/E5X, U302 AP22653AW6, U401 AP22653AW6, U402 MCP6486U, U403 IS31AP4991A-SLS2, U501 TPS7A2028PDBVR, U502 DPS310XTSA1, U503 HDC3022, U504 VL6180V1NR1, U601 TMUX1574RSV, U602 TMUX1574RSV, U603 TMUX1574RSV

Commit message: Added footprints for the TFTs we'll be using as eyes.
Parts:
- added EYE-LEFT: er-tft1.32-1-eye, msf-owl-clock:er-tft1.32-1-eye, F.Cu at (122.0, 64.0)
- added EYE-RIGHT: er-tft1.32-1-eye, msf-owl-clock:er-tft1.32-1-eye, F.Cu at (78.0, 64.0)
- LED001, Q301, R016, R017, R602, R603, R604, R605, R606, R607, R608, R609, R610, R611, R612, R613, U601, U602: moved to B.Cu
- moved C602 329.2 mm to (100.9, 83.2), turned to -90 degrees
- moved R611 326.9 mm to (98.7, 72.0), turned to 180 degrees
- moved R612 326.9 mm to (98.7, 74.0), turned to 180 degrees
- moved R613 326.9 mm to (98.7, 76.0), turned to 180 degrees
- moved C601 325.2 mm to (104.7, 83.2), turned to -90 degrees
- moved U602 323.7 mm to (100.3, 83.2), turned to 180 degrees
- moved R606 321.1 mm to (101.6, 72.0), turned to 180 degrees
- moved R607 321.1 mm to (101.6, 74.0), turned to 180 degrees
- moved R608 321.1 mm to (101.6, 76.0), turned to 180 degrees
- moved R609 321.1 mm to (101.6, 78.0), turned to 180 degrees
- moved R610 321.1 mm to (101.6, 80.0), turned to 180 degrees
- moved U601 316.2 mm to (104.1, 83.2), turned to 180 degrees
- moved R602 315.4 mm to (104.5, 74.0), turned to 180 degrees
- moved R603 315.4 mm to (104.5, 76.0), turned to 180 degrees
- moved R604 315.4 mm to (104.5, 78.0), turned to 180 degrees
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Routing:
- net GND: vias 53 -> 55
- net /CORE_VDD_{+3.3V}: vias 6 -> 8
Other:
- board text added: "PCB Capabilities: https://jlcpcb.com/capabilities/pcb-capabilities Tooling Holes: https://jlcpcb.com/help/article/47-How-to-add-tooling-holes-for-PCB-assembly-order"
- board text removed: "Tooling Holes: https://jlcpcb.com/help/article/47-How-to-add-tooling-holes-for-PCB-assembly-order"

Commit message: Finalised the location and dimensions of the eyes and their connectors; based on bench measurements.
Parts:
- CONN005, CONN006: moved to B.Cu
- moved CONN006 275.8 mm to (77.9, 66.5), turned to 180 degrees
- moved CONN005 231.6 mm to (122.1, 61.5)
Other:
- board text removed: "TODO: EYES ARE PLACED *ROUGHLY* - USE EXACT MEASUREMENTS FROM CENTRE LINE (100,100) WHEN PLACING THE TFTs"

Commit message: Added tie-wrap holes for the talons, along with a 3D model of the tie-wraps.
Parts:
- added TALON-LEFT: talon, msf-owl-clock:talon, F.Cu at (124.0, 181.5)
- added TALON-RIGHT: talon, msf-owl-clock:talon, F.Cu at (76.0, 181.5)
Other:
- board text removed: "TODO: PLACE THE HOLES (2x (3x 2.5mm TIE-WRAPS)) SLIGHTLY BEHIND THE FERRITE BAR, OR LEVEL WITH THE TOP OF ? WHICH ONE WILL FIT THE CURVE OF THE TIE-WRAPS BETTER AND LOOK BETTER ?"
Changed lines of the file:
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@@
     )
   )
+  (footprint "msf-owl-clock:talon" (layer "F.Cu")
+    (at 124 181.5)
+    (descr "Cut-Outs for Tie-Wraps - Serves as Talons")
+    (tags "owl-msf owl msf tie-wrap tie-wraps tiewrap tiewraps tie wrap wraps talon talons")
+    (attr through_hole board_only exclude_from_pos_files exclude_from_bom allow_missing_courtyard)
+    (fp_text reference "TALON-LEFT" (at 0 -2.4) (layer "F.SilkS") hide
+        (effects (font (size 1 1) (thickness 0.15)))
+    )
+    (fp_text value "talon" (at 0 2.2) (layer "F.Fab")
+        (effects (font (size 1 1) (thickness 0.15)))
+    )
+    (fp_text user "${REFERENCE}" (at 0 0) (layer "F.Fab")
+        (effects (font (size 0.98 0.98) (thickness 0.15)))
+    )
+    (pad "" np_thru_hole oval (at -7.5 -6.125) (size 3.75 1.25) (drill oval 3.75 1.25) (layers "F&B.Cu" "*.Mask"))
+    (pad "" np_thru_hole oval (at -7.5 6.125) (size 3.75 1.25) (drill oval 3.75 1.25) (layers "F&B.Cu" "*.Mask"))
+    (pad "" np_thru_hole oval (at 0 -6.125) (size 3.75 1.25) (drill oval 3.75 1.25) (layers "F&B.Cu" "*.Mask"))
+    (pad "" np_thru_hole oval (at 0 6.125) (size 3.75 1.25) (drill oval 3.75 1.25) (layers "F&B.Cu" "*.Mask"))
+    (pad "" np_thru_hole oval (at 7.5 -6.125) (size 3.75 1.25) (drill oval 3.75 1.25) (layers "F&B.Cu" "*.Mask"))
+    (pad "" np_thru_hole oval (at 7.5 6.125) (size 3.75 1.25) (drill oval 3.75 1.25) (layers "F&B.Cu" "*.Mask"))
+    (model "${KIPRJMOD}/msf-owl-clock.pretty/talon.step"
+      (offset (xyz -7.5 0 2.6))
+      (scale (xyz 1 1 1))
+      (rotate (xyz 90 0 0))
+    )
+  )
   (footprint "restall-generic-capacitors:unpolarised-nominal-0805-2012" (layer "F.Cu")
     (at 335.81 102.42)
@@
     )
   )
+  (footprint "msf-owl-clock:talon" (layer "F.Cu")
+    (at 76 181.5)
+    (descr "Cut-Outs for Tie-Wraps - Serves as Talons")
+    (tags "owl-msf owl msf tie-wrap tie-wraps tiewrap tiewraps tie wrap wraps talon talons")
+    (attr through_hole board_only exclude_from_pos_files exclude_from_bom allow_missing_courtyard)
+    (fp_text reference "TALON-RIGHT" (at 0 -2.4) (layer "F.SilkS") hide
+        (effects (font (size 1 1) (thickness 0.15)))
+    )
+    (fp_text value "talon" (at 0 2.2) (layer "F.Fab")
+        (effects (font (size 1 1) (thickness 0.15)))
+    )
+    (fp_text user "${REFERENCE}" (at 0 0) (layer "F.Fab")
+        (effects (font (size 0.98 0.98) (thickness 0.15)))
+    )
+    (pad "" np_thru_hole oval (at -7.5 -6.125) (size 3.75 1.25) (drill oval 3.75 1.25) (layers "F&B.Cu" "*.Mask"))
+    (pad "" np_thru_hole oval (at -7.5 6.125) (size 3.75 1.25) (drill oval 3.75 1.25) (layers "F&B.Cu" "*.Mask"))
+    (pad "" np_thru_hole oval (at 0 -6.125) (size 3.75 1.25) (drill oval 3.75 1.25) (layers "F&B.Cu" "*.Mask"))
+    (pad "" np_thru_hole oval (at 0 6.125) (size 3.75 1.25) (drill oval 3.75 1.25) (layers "F&B.Cu" "*.Mask"))
+    (pad "" np_thru_hole oval (at 7.5 -6.125) (size 3.75 1.25) (drill oval 3.75 1.25) (layers "F&B.Cu" "*.Mask"))
+    (pad "" np_thru_hole oval (at 7.5 6.125) (size 3.75 1.25) (drill oval 3.75 1.25) (layers "F&B.Cu" "*.Mask"))
+    (model "${KIPRJMOD}/msf-owl-clock.pretty/talon.step"
+      (offset (xyz -7.5 0 2.6))
+      (scale (xyz 1 1 1))
+      (rotate (xyz 90 0 0))
+    )
+  )
   (footprint "restall-generic-resistors:nominal-0402-1005" (layer "F.Cu")
     (at 336.41 128.9)
@@
   (gr_line locked (start 46.438013 147.054717) (end 45.431775 145.916333)
     (stroke (width 0.2) (type solid)) (layer "Edge.Cuts"))
-  (gr_text "TODO: PLACE THE HOLES (2x (3x 2.5mm TIE-WRAPS)) SLIGHTLY BEHIND THE FERRITE BAR, OR LEVEL WITH THE TOP OF ?  WHICH ONE WILL FIT THE CURVE OF THE TIE-WRAPS BETTER AND LOOK BETTER ?" (at 100 178) (layer "Cmts.User")
-    (effects (font (size 1 1) (thickness 0.15)))
-  )
   (gr_text "PCB Capabilities:\nhttps://jlcpcb.com/capabilities/pcb-capabilities\n\nTooling Holes:\nhttps://jlcpcb.com/help/article/47-How-to-add-tooling-holes-for-PCB-assembly-order" (at 199.9 22) (layer "F.Fab")
     (effects (font (size 1 1) (thickness 0.15)) (justify left bottom))

Commit message: PCB routing.
Parts:
- C309: moved to F.Cu
- moved C337 199.9 mm to (102.8, 94.2), turned to 90 degrees
- moved C338 196.9 mm to (106.2, 92.8)
- moved C339 193.3 mm to (110.2, 92.8), turned to 180 degrees
- moved C342 187.1 mm to (115.4, 107.2)
- moved C340 186.5 mm to (117.2, 94.1), turned to -90 degrees
- moved C341 186.0 mm to (117.2, 99.8), turned to 90 degrees
- moved U602 8.54 mm to (107.9, 87.1), turned to 90 degrees
- moved C602 8.32 mm to (107.9, 87.7), turned to 180 degrees
- moved C309 5.23 mm to (109.2, 107.2)
- moved C601 4.67 mm to (103.5, 87.7), turned to 180 degrees
- moved U601 3.94 mm to (103.5, 87.1), turned to 90 degrees
Connections:
- R604 pad 1: /6-tft-driver/TFT1.L_{IO3} -> /6-tft-driver/TFT1.L_{SDIN}
- R605 pad 1: /6-tft-driver/TFT0.L_{IO3} -> /6-tft-driver/TFT0.L_{SDIN}
- R606 pad 1: /6-tft-driver/TFT1.L_{SCLK} -> /6-tft-driver/TFT1.L_{IO1}
- R607 pad 1: /6-tft-driver/TFT0.L_{SCLK} -> /6-tft-driver/TFT0.L_{IO1}
- R608 pad 1: /6-tft-driver/TFT1.L_{SDIN} -> /6-tft-driver/TFT1.L_{IO3}
- R609 pad 1: /6-tft-driver/TFT0.L_{SDIN} -> /6-tft-driver/TFT0.L_{IO3}
- R612 pad 1: /6-tft-driver/TFT1.L_{IO1} -> /6-tft-driver/TFT1.L_{SCLK}
- R613 pad 1: /6-tft-driver/TFT0.L_{IO1} -> /6-tft-driver/TFT0.L_{SCLK}
- U601 pad 1: /6-tft-driver/TFT1.L_{SDIN} -> /6-tft-driver/TFT1.L_{IO3}
- U601 pad 16: /6-tft-driver/TFT0.L_{SDIN} -> /6-tft-driver/TFT0.L_{IO3}
- U601 pad 2: /3-mcu-core/DATA0 -> /3-mcu-core/DATA3
- U601 pad 3: /6-tft-driver/TFT0.L_{SCLK} -> /6-tft-driver/TFT0.L_{IO1}
- U601 pad 4: /6-tft-driver/TFT1.L_{SCLK} -> /6-tft-driver/TFT1.L_{IO1}
- U601 pad 5: /3-mcu-core/SCK -> /3-mcu-core/DATA1
- U601 pad 7: /3-mcu-core/DATA3 -> /3-mcu-core/DATA0
- U601 pad 8: /6-tft-driver/TFT1.L_{IO3} -> /6-tft-driver/TFT1.L_{SDIN}
- U601 pad 9: /6-tft-driver/TFT0.L_{IO3} -> /6-tft-driver/TFT0.L_{SDIN}
- U602 pad 3: /6-tft-driver/TFT0.L_{IO1} -> GND
- U602 pad 4: /6-tft-driver/TFT1.L_{IO1} -> GND
- U602 pad 5: /3-mcu-core/DATA1 -> GND
- U602 pad 7: GND -> /3-mcu-core/SCK
- U602 pad 8: GND -> /6-tft-driver/TFT1.L_{SCLK}
- U602 pad 9: GND -> /6-tft-driver/TFT0.L_{SCLK}
Routing:
- net /6-tft-driver/TFT0.L_{IO3}: track 0.00 -> 5.15 mm
- net /3-mcu-core/DATA0: track 0.00 -> 4.47 mm
- net /3-mcu-core/SCK: track 0.00 -> 3.77 mm
- net Net-(U301-PC20): track 0.00 -> 3.54 mm
- net /3-mcu-core/~{HMD_ALERT}: track 4.22 -> 0.96 mm
- net /3-mcu-core/DATA1: track 0.00 -> 2.87 mm
- net /3-mcu-core/DATA3: track 0.00 -> 2.75 mm
- net Net-(U301-PB14): track 0.00 -> 2.15 mm
- net /3-mcu-core/TFT_TEAR0: track 0.00 -> 1.66 mm, vias 0 -> 1
- net Net-(U301-PB15): track 0.00 -> 1.65 mm
- net /3-mcu-core/~{BAR_INT}: track 3.21 -> 1.66 mm
- net /3-mcu-core/PRX_GPIO0: track 2.37 -> 0.96 mm
- net /6-tft-driver/TFT1.L_{IO3}: track 0.00 -> 1.37 mm, vias 0 -> 1
- net /6-tft-driver/TFT1.L_{IO1}: track 0.00 -> 0.98 mm, vias 0 -> 1
- net /6-tft-driver/TFT0.L_{IO1}: track 0.00 -> 0.98 mm, vias 0 -> 1
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
Commit message: PCB routing.
Parts:
- C004, C005, C006, C007, C008, C009, C326, C327, C604, C605, Q602, Q603, R014, R329, R330, R331, R332, R333, R334, R335, R346, R347, R619, R620, U302: moved to B.Cu
- moved C605 354.0 mm to (78.7, 69.5), turned to -90 degrees
- moved Q603 351.0 mm to (83.7, 67.1)
- moved R620 347.0 mm to (83.7, 65.2), turned to 180 degrees
- moved Q602 319.6 mm to (116.3, 60.9), turned to 180 degrees
- moved R619 315.1 mm to (116.3, 62.8)
- moved C604 314.0 mm to (121.3, 58.5), turned to 90 degrees
- moved C009 300.8 mm to (75.8, 69.5), turned to -90 degrees
- moved C008 296.0 mm to (77.7, 69.5), turned to -90 degrees
- moved C007 294.0 mm to (79.7, 69.5), turned to -90 degrees
- moved C006 253.4 mm to (120.3, 58.5), turned to 90 degrees
- moved C005 248.7 mm to (122.3, 58.5), turned to 90 degrees
- moved C004 246.7 mm to (124.2, 58.5), turned to 90 degrees
- moved R014 224.4 mm to (122.3, 96.7), turned to 180 degrees
- moved R332 203.0 mm to (119.7, 97.0)
- moved R335 200.6 mm to (122.3, 93.4)
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Routing:
- net /6-tft-driver/TFT1.L_{SCLK}: track 0.00 -> 48.9 mm
- net /6-tft-driver/TFT0.L_{SCLK}: track 0.00 -> 31.9 mm
- net /6-tft-driver/TFT0.~{L_{RES}}: track 0.00 -> 24.9 mm
- net /CORE_VDD_{+3.3V}: track 8.36 -> 32.7 mm, vias 16 -> 23
- net /3-mcu-core/TFT_BACKLED1: track 0.00 -> 19.1 mm
- net /3-mcu-core/TFT_BACKLED0: track 0.00 -> 15.4 mm
- net /6-tft-driver/TFT1.~{L_{RES}}: track 0.00 -> 14.5 mm
- net /3-mcu-core/BC805M.~{CTS}: track 0.00 -> 13.0 mm
- net /3-mcu-core/BC805M.SWDIO: track 0.00 -> 13.0 mm
- net /3-mcu-core/BC805M.SCK: track 0.00 -> 12.8 mm
- net /6-tft-driver/TFT1.~{TP_{RST}}: track 0.00 -> 12.5 mm
- net /6-tft-driver/TFT0.~{TP_{RST}}: track 0.00 -> 12.5 mm
- net /6-tft-driver/TFT0.LED_{A}: track 0.00 -> 12.3 mm
- net /3-mcu-core/BC805M.SWDCLK: track 0.00 -> 11.9 mm
- net /6-tft-driver/TFT1.LED_{A}: track 0.00 -> 11.7 mm
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Other:
- board text added: "TODO: EYES SOLDERMASK OVER VIAS NO TRACKS ON TOP LAYER"

Commit message: PCB routing.
Parts:
- C218, C219, C220, C221, C222, C223, C224, C225, C226, C227, C228, C229, C233, C234, C235, C236, C237, C238, C243, D201, D202, D203, D204, D205, NT201, R201, R202, R203, R204, R205, R206, R207, R208, R209, R210, R211, R225, R226, R227, R228, R229, R230, R231, R232, R233, R234, TP203, TP204, TP207, U203, U206: moved to B.Cu
- moved NT201 440.4 mm to (-56.9, 160.1), turned to 180 degrees
- moved C233 432.0 mm to (-52.7, 170.2), turned to 180 degrees
- moved C234 432.0 mm to (-52.7, 172.2), turned to 180 degrees
- moved TP207 410.4 mm to (-41.8, 170.6), turned to 180 degrees
- moved C238 393.1 mm to (-13.0, 150.9), turned to -90 degrees
- moved D202 392.1 mm to (-46.9, 121.3), turned to 180 degrees
- moved D203 392.1 mm to (-46.9, 124.2), turned to 180 degrees
- moved D205 392.1 mm to (-46.9, 130.1), turned to 180 degrees
- moved C236 391.0 mm to (-10.7, 151.4), turned to 180 degrees
- moved TP203 390.6 mm to (-46.1, 141.3), turned to 180 degrees
- moved TP204 390.6 mm to (-46.1, 144.0), turned to 180 degrees
- moved C237 389.8 mm to (-8.70, 151.4), turned to -90 degrees
- moved C243 385.7 mm to (-1.80, 151.0)
- moved R233 384.9 mm to (-14.2, 151.9), turned to -90 degrees
- moved R234 384.9 mm to (-14.2, 153.8), turned to -90 degrees
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Connections:
- U206 pad 12: GND -> unconnected-(U206E-NC-Pad7)
- U206 pad 7: GND -> unconnected-(U206E-NC-Pad7)
- U207 pad 7: GND -> unconnected-(U207E-NC-Pad7)
Routing:
- net /2-msf-receiver/MSF_RCV_VREF_{+1.8V}: track 0.00 -> 22.8 mm
- net /2-msf-receiver/2-msf-receiver-trf/PGA1.SW_EN3: track 0.00 -> 10.3 mm
- net /2-msf-receiver/MSF_RCV_VREF_{+2.5V}: track 0.00 -> 7.85 mm
- net Net-(U203D--): track 0.00 -> 6.92 mm
- net /2-msf-receiver/2-msf-receiver-trf/PGA1.FB3: track 0.00 -> 6.32 mm
- net /2-msf-receiver/2-msf-receiver-trf/PGA1.FB4: track 0.00 -> 5.46 mm
- net Net-(U203C--): track 0.00 -> 4.93 mm
- net Net-(U203B--): track 0.00 -> 4.93 mm
- net Net-(C225-Pad2): track 0.00 -> 4.92 mm
- net Net-(C219-Pad2): track 0.00 -> 4.81 mm
- net /2-msf-receiver/2-msf-receiver-trf/MSF_RCV_TRF1: track 0.00 -> 4.47 mm
- net /2-msf-receiver/2-msf-receiver-trf/PGA1.SW_EN2: track 0.00 -> 4.47 mm
- net /2-msf-receiver/2-msf-receiver-trf/PGA1.SW_EN1: track 0.00 -> 4.25 mm
- net /2-msf-receiver/2-msf-receiver-trf/PGA1.FB0: track 0.00 -> 4.17 mm
- net /2-msf-receiver/2-msf-receiver-trf/PGA1.FB1: track 0.00 -> 4.03 mm
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