File: src/schematics/6-tft-driver.kicad_sch (KiCad schematic)
At the start: 41 parts, among them Q601 NX6008NBKW, Q602 BC847BS, Q603 BC847BS, U601 TMUX1574RSV, U602 TMUX1574RSV, U603 TMUX1574RSV

Commit message: PCB routing.
Parts:
- removed NT609, NT610: Net Tie, restall-generic-wires:net-tie-2-6mil, symbol restall-generic-wires:net-tie-2
Connections:
- net TFT0.LED_{A} is gone; now on net CORE_VDD_{+5V}: C604.1
- net TFT1.LED_{A} is gone; now on net CORE_VDD_{+5V}: C605.1
Changed lines of the file:
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@@
     (stroke (width 0) (type default))
   )
-  (wire (pts (xy 111.76 226.06) (xy 119.38 226.06))
-    (stroke (width 0) (type default))
-  )
-  (wire (pts (xy 68.58 226.06) (xy 76.2 226.06))
+  (wire (pts (xy 109.22 226.06) (xy 119.38 226.06))
+    (stroke (width 0) (type default))
+  )
+  (wire (pts (xy 66.04 226.06) (xy 76.2 226.06))
     (stroke (width 0) (type default))
   )
@@
     )
   )
-  (symbol (lib_id "restall-generic-wires:net-tie-2") (at 110.49 226.06 0) (unit 1)
-    (in_bom no) (on_board yes) (dnp no) (fields_autoplaced)
-    (property "Reference" "NT610" (at 110.49 223.52 0)
-      (effects (font (size 1.27 1.27)) hide)
-    )
-    (property "Value" "Net Tie" (at 110.49 228.6 0)
-      (effects (font (size 1.27 1.27)) hide)
-    )
-    (property "Footprint" "restall-generic-wires:net-tie-2-6mil" (at 110.49 230.632 0)
-      (effects (font (size 1.27 1.27)) hide)
-    )
-    (property "Datasheet" "~" (at 110.49 232.664 0)
-      (effects (font (size 1.27 1.27)) hide)
-    )
-    (pin "2" (alternate "P2_PWROUT"))
-    (pin "1" (alternate "P1_PWRIN"))
-    (instances
-      (project "msf-owl-clock"
-        (path "/56d623d3-22db-4d43-a9d9-e6bb4bb68946/2680f60f-7a4f-44d1-82ff-576d0b59662d"
-          (reference "NT610") (unit 1)
-        )
-      )
-    )
-  )
   (symbol (lib_id "restall-generic-wires:net-tie-2") (at 81.28 153.67 270) (unit 1)
     (in_bom no) (on_board yes) (dnp no) (fields_autoplaced)
@@
         )
       )
-    )
-  )
-  (symbol (lib_id "restall-generic-wires:net-tie-2") (at 67.31 226.06 0) (unit 1)
-    (in_bom no) (on_board yes) (dnp no) (fields_autoplaced)
-    (property "Reference" "NT609" (at 67.31 223.52 0)
-      (effects (font (size 1.27 1.27)) hide)
-    )
-    (property "Value" "Net Tie" (at 67.31 228.6 0)
-      (effects (font (size 1.27 1.27)) hide)
-    )
-    (property "Footprint" "restall-generic-wires:net-tie-2-6mil" (at 67.31 230.632 0)
-      (effects (font (size 1.27 1.27)) hide)
-    )
-    (property "Datasheet" "~" (at 67.31 232.664 0)
-      (effects (font (size 1.27 1.27)) hide)
-    )
-    (pin "2" (alternate "P2_PWROUT"))
-    (pin "1" (alternate "P1_PWRIN"))
-    (instances
-      (project "msf-owl-clock"
-        (path "/56d623d3-22db-4d43-a9d9-e6bb4bb68946/2680f60f-7a4f-44d1-82ff-576d0b59662d"
-          (reference "NT609") (unit 1)
-        )
-      )

Commit message: PCB routing.
Changed lines of the file:
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@@
     (stroke (width 0) (type default))
   )
-  (wire (pts (xy 60.96 52.07) (xy 60.96 53.086))
+  (wire (pts (xy 60.96 52.07) (xy 60.96 53.34))
     (stroke (width 0) (type default))
   )
@@
     (stroke (width 0) (type default))
   )
-  (wire (pts (xy 60.96 63.246) (xy 60.96 63.5))
-    (stroke (width 0) (type default))
-  )
   (bus (pts (xy 88.9 223.52) (xy 88.9 231.14))
     (stroke (width 0) (type default))
@@
   )
   (wire (pts (xy 327.66 73.66) (xy 360.68 73.66))
-    (stroke (width 0) (type default))
-  )
-  (wire (pts (xy 53.34 58.166) (xy 53.34 58.42))
     (stroke (width 0) (type default))
   )
@@
     )
   )
-  (symbol (lib_id "restall-manufacturer-nexperia:NX6008NBKW") (at 58.42 58.166 0) (unit 1)
+  (symbol (lib_id "restall-manufacturer-nexperia:NX6008NBKW") (at 58.42 58.42 0) (unit 1)
     (in_bom yes) (on_board yes) (dnp no)
-    (property "Reference" "Q601" (at 63.5 56.134 0)
-      (effects (font (size 1.27 1.27)) (justify left))
-    )
-    (property "Value" "NX6008NBKW" (at 63.5 58.166 0)
-      (effects (font (size 1.27 1.27)) (justify left))
-    )
-    (property "Footprint" "restall-generic-sot:SOT323" (at 63.5 54.61 0)
-      (effects (font (size 1.27 1.27)) (justify left) hide)
-    )
-    (property "Datasheet" "https://assets.nexperia.com/documents/data-sheet/NX6008NBKW.pdf" (at 63.5 66.294 0)
-      (effects (font (size 1.27 1.27)) (justify left) hide)
-    )
-    (property "Package" "SOT323" (at 63.5 60.198 0)
-      (effects (font (size 1.27 1.27)) (justify left))
-    )
-    (property "Manufacturer" "Nexperia" (at 63.5 64.008 0)
-      (effects (font (size 1.27 1.27)) (justify left) hide)
-    )
-    (property "ManufacturerPartNumber" "NX6008NBKW" (at 63.5 61.722 0)
-      (effects (font (size 1.27 1.27)) (justify left) hide)
-    )
+    (property "Reference" "Q601" (at 63.5 56.388 0)
+      (effects (font (size 1.27 1.27)) (justify left))
+    )
+    (property "Value" "NX6008NBKW" (at 63.5 58.42 0)
+      (effects (font (size 1.27 1.27)) (justify left))
+    )
+    (property "Footprint" "restall-generic-sot:SOT323" (at 63.5 54.864 0)
+      (effects (font (size 1.27 1.27)) (justify left) hide)
+    )
+    (property "Datasheet" "https://assets.nexperia.com/documents/data-sheet/NX6008NBKW.pdf" (at 63.5 66.548 0)
+      (effects (font (size 1.27 1.27)) (justify left) hide)
+    )
+    (property "Package" "SOT323" (at 63.5 60.452 0)
+      (effects (font (size 1.27 1.27)) (justify left))
+    )
+    (property "Manufacturer" "Nexperia" (at 63.5 64.262 0)
+      (effects (font (size 1.27 1.27)) (justify left) hide)
+    )
+    (property "ManufacturerPartNumber" "NX6008NBKW" (at 63.5 61.976 0)
+      (effects (font (size 1.27 1.27)) (justify left) hide)
+    )
